File: hardware/programmer/programmer.kicad_pcb (KiCad board)
At the start: 2 copper layers, 32 parts, among them SW1 SW_Push, SW2 SW_Push, U2 NCP1117-3.3_SOT223, U5 W25Q128JVS, Y1 ABM8-272-T3

Commit message: Update
Parts:
- removed R10: 0, Resistor_SMD:R_0402_1005Metric
- removed R9: DNF, Resistor_SMD:R_0402_1005Metric
- added C6: 4.7u, Capacitor_SMD:C_0402_1005Metric, F.Cu at (148.0, 127.7)
- added C7: 4.7u, Capacitor_SMD:C_0402_1005Metric, F.Cu at (148.0, 126.8)
- added H1: MountingHole, MountingHole:MountingHole_3.2mm_M3, F.Cu at (127.7, 156.4)
- added H2: MountingHole, MountingHole:MountingHole_3.2mm_M3, F.Cu at (167.7, 116.4)
- added H3: MountingHole, MountingHole:MountingHole_3.2mm_M3, F.Cu at (127.7, 116.4)
- added H4: MountingHole, MountingHole:MountingHole_3.2mm_M3, F.Cu at (167.7, 156.4)
- added J1: Micro_SD_Card, inkbadge:SDCardlcsc, F.Cu at (162.0, 129.2)
- added J2: USB_C_Receptacle_USB2.0_14P, Connector_USB:USB_C_Receptacle_GCT_USB4105-xx-A_16P_TopMnt_Horizontal, F.Cu at (145.7, 116.1)
- added J3: Bus_PCI_Express_x4, programmer:PCIe_x4_Edgeboard_Connector, F.Cu at (140.2, 146.8)
- added L1: 3.3u, Inductor_SMD:L_Cenker_CKCS201610, F.Cu at (148.0, 125.0)
- R3, R5: value DNF -> 5.1k
- moved C16 43.8 mm to (143.9, 137.8), turned to -90 degrees
- moved C3 43.7 mm to (141.9, 140.7), turned to 90 degrees
- moved C4 40.9 mm to (147.1, 140.7), turned to -90 degrees
- moved C12 39.7 mm to (148.8, 137.3), turned to -90 degrees
- moved R2 39.5 mm to (145.4, 137.6), turned to -90 degrees
- moved U1 36.9 mm to (146.0, 132.3)
- moved R4 35.7 mm to (147.8, 137.7), turned to -90 degrees
- moved C11 35.6 mm to (151.6, 131.6)
- moved R6 35.4 mm to (136.2, 129.2), turned to -90 degrees
- moved C17 35.3 mm to (140.9, 129.4), turned to 180 degrees
- moved C10 34.4 mm to (146.3, 138.0), turned to -90 degrees
- moved C15 32.5 mm to (140.9, 133.5), turned to 180 degrees
- moved C8 31.6 mm to (140.3, 131.5), turned to 180 degrees
- moved C14 30.7 mm to (151.6, 132.6)
- moved SW1 29.9 mm to (137.3, 132.6), turned to 90 degrees
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Connections:
- R1 pad 2: /FLASH_SS -> /QSPI_SS
- R7 pad 1: /USB_D+ -> /D+
- R8 pad 1: /USB_D- -> /D-
- U1 pad 32: unconnected-(U1-GPIO20-Pad32) -> /MISO
- U1 pad 33: unconnected-(U1-GPIO21-Pad33) -> /CS
- U1 pad 34: unconnected-(U1-GPIO22-Pad34) -> /CLK
- U1 pad 35: unconnected-(U1-GPIO23-Pad35) -> /MOSI
- U1 pad 36: unconnected-(U1-GPIO24-Pad36) -> /MISO1
- U1 pad 37: unconnected-(U1-GPIO25-Pad37) -> /SDCS
- U1 pad 40: unconnected-(U1-GPIO26_ADC0-Pad40) -> /SCLK1
- U1 pad 41: unconnected-(U1-GPIO27_ADC1-Pad41) -> /MOSI1
- U5 pad 1: /FLASH_SS -> /QSPI_SS
Routing:
- net +5V: track 0.00 -> 67.7 mm
- net +3V3: track 0.00 -> 58.5 mm, vias 0 -> 5
- net /MOSI: track 0.00 -> 22.3 mm
- net /QSPI_SS: track 0.00 -> 21.6 mm
- net /MISO: track 0.00 -> 20.1 mm
- net /CS: track 0.00 -> 19.1 mm
- net /CLK: track 0.00 -> 18.3 mm
- net +1V1: track 0.00 -> 17.1 mm, vias 0 -> 9
- net /SDCS: track 0.00 -> 12.2 mm, vias 0 -> 2
- net /QSPI_SD1: track 0.00 -> 12.1 mm
- net /QSPI_SD2: track 0.00 -> 9.00 mm
- net /XIN: track 0.00 -> 8.12 mm
- net /D+: track 0.00 -> 7.02 mm
- net GND: track 0.00 -> 6.33 mm, vias 0 -> 33
- net /D-: track 0.00 -> 6.08 mm
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- added copper zone on F.Cu, net +1V1
- added copper zone on F.Cu, net +3V3
- added copper zone on F.Cu, net +5V
- added copper zone on F.Cu, net /VREG_LX
- added copper zone on B.Cu, net GND
- added copper zone on F.Cu, net GND
Other:
- board outline added: 50 x 50 mm

Commit message: Finish programmer
Parts:
- added U3: SRV05-4, Package_TO_SOT_SMD:SOT-23-6, F.Cu at (146.0, 123.4)
- H1, H2, H3, H4: footprint MountingHole:MountingHole_3.2mm_M3 -> MountingHole:MountingHole_2.2mm_M2_Pad_Via
- Y1: value ABM8-272-T3 -> 12MHz 10pf; footprint Crystal:Crystal_SMD_3225-4Pin_3.2x2.5mm -> Crystal:Crystal_SMD_2520-4Pin_2.5x2.0mm
- moved R1 6.25 mm to (137.7, 124.2)
- moved J3 4.47 mm to (142.9, 150.3)
- moved C2 3.35 mm to (141.8, 124.2)
- moved Y1 2.56 mm to (145.4, 143.1)
- moved C11 2.15 mm to (151.6, 133.8)
- moved C13 2.15 mm to (151.0, 131.8)
- moved C15 2.15 mm to (140.9, 135.7)
- moved C17 2.15 mm to (140.9, 131.6)
- moved C5 2.15 mm to (162.6, 119.0)
- moved C6 2.15 mm to (148.0, 129.9)
- moved C8 2.15 mm to (140.3, 133.7)
- moved J1 2.15 mm to (162.0, 131.4)
- moved R4 2.15 mm to (147.8, 139.8)
- moved R6 2.15 mm to (136.2, 131.4)
- moved R7 2.15 mm to (145.1, 127.1)
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Connections:
- J3 pad A5: unconnected-(J3-JTAG2-PadA5) -> /CLK
- J3 pad A6: unconnected-(J3-JTAG3-PadA6) -> /MOSI
- J3 pad A7: unconnected-(J3-JTAG4-PadA7) -> /MISO
- J3 pad A8: unconnected-(J3-JTAG5-PadA8) -> /CS
- J3 pad B14: /MISO -> unconnected-(J3-PETp0-PadB14)
- J3 pad B15: /CS -> unconnected-(J3-PETn0-PadB15)
- J3 pad B19: /CLK -> unconnected-(J3-PETp1-PadB19)
- J3 pad B20: /MOSI -> unconnected-(J3-PETn1-PadB20)
- J3 pad B5: unconnected-(J3-SMCLK-PadB5) -> /I2C_CLK
- J3 pad B6: unconnected-(J3-SMDAT-PadB6) -> /I2C_DATA
- U1 pad 12: unconnected-(U1-GPIO8-Pad12) -> /MISO
- U1 pad 13: unconnected-(U1-GPIO9-Pad13) -> /CS
- U1 pad 14: unconnected-(U1-GPIO10-Pad14) -> /CLK
- U1 pad 15: unconnected-(U1-GPIO11-Pad15) -> /MOSI
- U1 pad 32: /MISO -> /MISO1
- U1 pad 33: /CS -> /SDCS
- U1 pad 34: /CLK -> /SCLK1
- U1 pad 35: /MOSI -> /MOSI1
- U1 pad 36: /MISO1 -> unconnected-(U1-GPIO24-Pad36)
- U1 pad 37: /SDCS -> unconnected-(U1-GPIO25-Pad37)
- U1 pad 40: /SCLK1 -> unconnected-(U1-GPIO26_ADC0-Pad40)
- U1 pad 41: /MOSI1 -> unconnected-(U1-GPIO27_ADC1-Pad41)
Routing:
- net /CS: track 19.1 -> 12.7 mm
- net +5V: track 67.7 -> 73.4 mm, vias 0 -> 2
- net /QSPI_SS: track 21.6 -> 16.0 mm
- net /MISO: track 20.1 -> 15.6 mm
- net +3V3: track 58.5 -> 62.2 mm
- net GND: track 6.33 -> 2.91 mm, vias 33 -> 46
- net /MOSI1: track 6.07 -> 8.85 mm
- net /D-: track 6.08 -> 8.83 mm
- net /D+: track 7.02 -> 9.28 mm
- net /MOSI: track 22.3 -> 24.1 mm
- net /SCLK1: track 5.38 -> 7.05 mm
- net /XIN: track 8.12 -> 7.08 mm
- net Net-(J2-CC2): track 2.57 -> 1.67 mm
- net +1V1: track 17.1 -> 16.3 mm
Other:
- board size 50 x 50 mm -> 50 x 49 mm

Commit message: SOME FIRMWARE IG FAQ THE WORLD IDC ME DIE
Parts:
- added C40: 4.7uF, Capacitor_SMD:C_0402_1005Metric, F.Cu at (150.4, 130.2)
- added G***: LOGO, LOGO, F.Cu at (135.7, 159.2)
- added G***: LOGO, LOGO, F.Cu at (129.6, 133.7)
- added G***: LOGO, LOGO, F.Cu at (160.4, 143.1)
- added G***: LOGO, LOGO, F.Cu at (129.6, 133.9)
- added G***: LOGO, LOGO, B.Cu at (115.5, 134.9)
- added G***: LOGO, LOGO, B.Cu at (158.9, 116.0)
- added R16: 33, Resistor_SMD:R_0402_1005Metric, F.Cu at (150.4, 129.3)
- C6, C7: footprint Capacitor_SMD:C_0402_1005Metric -> rp2350:C_0402_1005Metric_small_pads
- L1: footprint Inductor_SMD:L_Cenker_CKCS201610 -> rp2350:L_pol_2016
- R1: value DNF -> 10k
- SW1, SW2: footprint Button_Switch_SMD:SW_SPST_B3U-1000P -> inkbadge:SW_Push_SPST_TSA016
- Y1: footprint Crystal:Crystal_SMD_2520-4Pin_2.5x2.0mm -> Crystal:Crystal_SMD_3225-4Pin_3.2x2.5mm
- moved H1 1.00 mm to (127.7, 157.4)
- moved H2 1.00 mm to (167.7, 117.4)
- moved H3 1.00 mm to (127.7, 117.4)
- moved H4 1.00 mm to (167.7, 157.4)
- moved SW2 0.45 mm to (149.9, 143.2), turned to -90 degrees
- moved R4 0.30 mm to (147.8, 139.6)
- moved Y1 0.25 mm to (145.4, 143.3)
- moved SW1 0.21 mm to (137.2, 134.9), turned to -90 degrees
Connections:
- H1 pad 1: (no net) -> GND
- H2 pad 1: (no net) -> GND
- H3 pad 1: (no net) -> GND
- H4 pad 1: (no net) -> GND
- U1 pad 46: unconnected-(U1-VREG_AVDD-Pad46) -> Net-(U1-VREG_AVDD)
Routing:
- net +3V3: track 62.2 -> 71.9 mm, vias 5 -> 6
- net /~{USB_BOOT}: track 1.62 -> 5.13 mm
- net Net-(R4-Pad2): track 2.66 -> 5.31 mm
- net Net-(U1-VREG_AVDD): track 0.00 -> 2.41 mm
- net GND: track 2.91 -> 3.53 mm, vias 46 -> 53
Other:
- board size 50 x 49 mm -> 50 x 50 mm
- board text added: "@ GitHub HQ San Francisco"
- board text added: "BOOT"
- board text added: "July 11 - 14"
- board text added: "RUN"
