File: hardware/programmer/programmer.kicad_sch (KiCad schematic)
At the start: 37 parts, among them J1 Micro_SD_Card, J2 USB_C_Receptacle_USB2.0_14P, SW1 SW_Push, SW2 SW_Push, U2 NCP1117-3.3_SOT223, U5 W25Q128JVS, Y1 ABM8-272-T3

Commit message: Update
Parts:
- removed R10: 0, Resistor_SMD:R_0402_1005Metric, symbol Device:R
- removed R9: DNF, Resistor_SMD:R_0402_1005Metric, symbol Device:R
- added H1, H2, H3, H4: MountingHole, MountingHole:MountingHole_3.2mm_M3, symbol Mechanical:MountingHole
- added J3: Bus_PCI_Express_x4, programmer:PCIe_x4_Edgeboard_Connector, symbol Connector:Bus_PCI_Express_x4
- C6, C7: footprint RP2350_60QFN_minimal:C_0402_1005Metric_small_pads -> Capacitor_SMD:C_0402_1005Metric
- J2: footprint (none) -> Connector_USB:USB_C_Receptacle_GCT_USB4105-xx-A_16P_TopMnt_Horizontal; LCSC Part # (none) -> C2765186
- L1: footprint RP2350_60QFN_minimal:L_pol_2016 -> Inductor_SMD:L_Cenker_CKCS201610
- R3, R5: value DNF -> 5.1k
Connections:
- net FLASH_SS is gone; now on net QSPI_SS: R1.2, U5.1 (~{CS})
- net SCLK is gone; now on net SCLK1: J1.5 (CLK)
- net USB_D+ is gone; now on net D+: R7.1
- net USB_D- is gone; now on net D-: R8.1
- net +3V3: now also J3.A10 (+3.3V), J3.A9 (+3.3V), J3.B10 (3.3Vaux), J3.B8 (+3.3V)
- net +5V: now also J3.A2 (+12V), J3.A3 (+12V), J3.B1 (+12V), J3.B2 (+12V), J3.B3 (+12V)
- net D+: now also J2.A6 (D+), J2.B6 (D+); no longer J2.A7 (D-), J2.B7 (D-)
- net D-: now also J2.A7 (D-), J2.B7 (D-); no longer J2.A6 (D+), J2.B6 (D+)
- net GND: now also J3.A12 (GND), J3.A15 (GND), J3.A18 (GND), J3.A20 (GND), J3.A23 (GND), J3.A24 (GND), J3.A27 (GND), J3.A28 (GND), J3.A31 (GND), J3.A4 (GND), J3.B13 (GND), J3.B16 (GND), J3.B18 (GND), J3.B21 (GND), J3.B22 (GND), J3.B25 (GND), J3.B26 (GND), J3.B29 (GND), J3.B32 (GND), J3.B4 (GND), J3.B7 (GND)
- net MISO: now also U1.32 (GPIO20), J3.B14 (PETp0); no longer J1.7 (DAT0)
- net MOSI: now also U1.35 (GPIO23), J3.B20 (PETn1); no longer J1.3 (CMD)
- net SDCS: now also U1.37 (GPIO25)
- net CS: now reaches U1.33 (GPIO21)
- net CS: now also J3.B15 (PETn0)
- net CLK: now reaches U1.34 (GPIO22)
- net CLK: now also J3.B19 (PETp1)
- net MISO1: now reaches U1.36 (GPIO24)
- net MISO1: now also J1.7 (DAT0)
- net SCLK1: now reaches U1.40 (GPIO26_ADC0)
- net MOSI1: now reaches U1.41 (GPIO27_ADC1)
- net MOSI1: now also J1.3 (CMD)
Other:
- note removed: "Make sure R7 and R8 are close to RP2350"
- moved on the sheet: C1, C10, C11, C12, C13, C14, C15, C16, C17, C18, C19, C2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

Commit message: Finish programmer
Parts:
- added U3: SRV05-4, Package_TO_SOT_SMD:SOT-23-6, symbol Power_Protection:SRV05-4
- H1, H2, H3, H4: footprint MountingHole:MountingHole_3.2mm_M3 -> MountingHole:MountingHole_2.2mm_M2_Pad_Via
- Y1: value ABM8-272-T3 -> 12MHz 10pf; footprint Crystal:Crystal_SMD_3225-4Pin_3.2x2.5mm -> Crystal:Crystal_SMD_2520-4Pin_2.5x2.0mm; LCSC Part # (none) -> C7301971
Connections:
- net +5V: now also U3.5 (VP)
- net CLK: now also J3.A5 (JTAG2), U1.14 (GPIO10); no longer J3.B19 (PETp1), U1.34 (GPIO22)
- net CS: now also J3.A8 (JTAG5), U1.13 (GPIO9); no longer J3.B15 (PETn0), U1.33 (GPIO21)
- net D+: now also U3.3 (IO2), U3.4 (IO3)
- net D-: now also U3.1 (IO1), U3.6 (IO4)
- net GND: now also U3.2 (VN)
- net MISO: now also J3.A7 (JTAG4), U1.12 (GPIO8); no longer J3.B14 (PETp0), U1.32 (GPIO20)
- net MISO1: now also U1.32 (GPIO20); no longer U1.36 (GPIO24)
- net MOSI: now also J3.A6 (JTAG3), U1.15 (GPIO11); no longer J3.B20 (PETn1), U1.35 (GPIO23)
- net MOSI1: now also U1.35 (GPIO23); no longer U1.41 (GPIO27_ADC1)
- net SCLK1: now also U1.34 (GPIO22); no longer U1.40 (GPIO26_ADC0)
- net SDCS: now also U1.33 (GPIO21); no longer U1.37 (GPIO25)
- net I2C_CLK: now reaches J3.B5 (SMCLK)
- net I2C_DATA: now reaches J3.B6 (SMDAT)
- no-connect marks 2 -> 21
Other:
- note added: "SPI1"
- moved on the sheet: C1, C10, C11, C12, C13, C14, C15, C16, C17, C18, C19, C5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

Commit message: SOME FIRMWARE IG FAQ THE WORLD IDC ME DIE
Parts:
- added C40: 4.7uF, Capacitor_SMD:C_0402_1005Metric, symbol Device:C
- added R16: 33, Resistor_SMD:R_0402_1005Metric, symbol Device:R
- C1, C19, C5: LCSC Part # (none) -> C19702
- C10: LCSC Part # (none) -> C23733
- C11, C12, C13, C14, C15, C16, C17, C18, C2, C8: LCSC Part # (none) -> C1525
- C3, C4: LCSC Part # (none) -> C1548
- C6, C7: footprint Capacitor_SMD:C_0402_1005Metric -> rp2350:C_0402_1005Metric_small_pads; LCSC Part # (none) -> C23733
- H1, H2, H3, H4: symbol Mechanical:MountingHole -> Mechanical:MountingHole_Pad
- J3: LCSC Part # (none) -> C2832353
- L1: footprint Inductor_SMD:L_Cenker_CKCS201610 -> rp2350:L_pol_2016; LCSC Part # (none) -> C42411119
- R1: value DNF -> 10k; LCSC Part # (none) -> C25744
- R2, R4, R6: LCSC Part # (none) -> C11702
- R3, R5: LCSC Part # (none) -> C25905
- R7, R8: LCSC Part # (none) -> C25105
- SW1, SW2: footprint Button_Switch_SMD:SW_SPST_B3U-1000P -> inkbadge:SW_Push_SPST_TSA016; LCSC Part # (none) -> C2888430
- U1: LCSC Part # (none) -> C42411118
- U2: LCSC Part # (none) -> C6186
- U3: LCSC Part # (none) -> C85364
- U5: LCSC Part # (none) -> C97521
- Y1: footprint Crystal:Crystal_SMD_2520-4Pin_2.5x2.0mm -> Crystal:Crystal_SMD_3225-4Pin_3.2x2.5mm; LCSC Part # C7301971 -> C20625731
Connections:
- net +3V3: now also R16.1
- net GND: now also H1.1, H2.1, H3.1, H4.1, C40.2
- net at U1.46 (VREG_AVDD): now also C40.1, R16.2
