File: inkbadge/inkbadge.kicad_pcb (KiCad board)
At the start: 2 copper layers, 38 parts, among them J4 USB_C_Receptacle_USB2.0_14P, SW1 SW_Push, SW2 SW_Push, U2 NCP1117-3.3_SOT223, U3 W25Q128JVS, Y1 ABM8-272-T3

Commit message: Progress
Parts:
- added C20: 1u, Capacitor_SMD:C_0402_1005Metric, F.Cu at (132.2, 95.5)
- added C21: 1u, Capacitor_SMD:C_0402_1005Metric, F.Cu at (132.2, 97.5)
- added C22: 1u, Capacitor_SMD:C_0402_1005Metric, F.Cu at (132.2, 99.5)
- added C23: 1u, Capacitor_SMD:C_0402_1005Metric, F.Cu at (132.2, 101.4)
- added C24: 1u, Capacitor_SMD:C_0402_1005Metric, F.Cu at (132.2, 103.4)
- added C25: 1u, Capacitor_SMD:C_0402_1005Metric, F.Cu at (135.1, 95.5)
- added C26: 1u, Capacitor_SMD:C_0402_1005Metric, F.Cu at (135.1, 97.5)
- added C27: 4.7uF, Capacitor_SMD:C_0402_1005Metric, F.Cu at (135.1, 99.5)
- added C28: 1u, Capacitor_SMD:C_0402_1005Metric, F.Cu at (135.1, 101.4)
- added C29: 4.7uF, Capacitor_SMD:C_0402_1005Metric, F.Cu at (135.1, 103.4)
- added C30: 1u, Capacitor_SMD:C_0402_1005Metric, F.Cu at (138.0, 95.5)
- added C31: 1u, Capacitor_SMD:C_0402_1005Metric, F.Cu at (138.0, 97.5)
- added C32: 10u, Capacitor_SMD:C_0402_1005Metric, F.Cu at (138.0, 99.5)
- added D1: MBR0530, Diode_SMD:D_SOD-123, F.Cu at (127.9, 96.2)
- added D2: MBR0530, Diode_SMD:D_SOD-123, F.Cu at (127.9, 99.6)
- added D3: MBR0530, Diode_SMD:D_SOD-123, F.Cu at (127.9, 102.9)
- added J1: Micro_SD_Card, inkbadge:SDCardlcsc, F.Cu at (151.5, 119.7)
- added Q1: Si1308EDL, Package_TO_SOT_SMD:SOT-323_SC-70, F.Cu at (133.0, 106.4)
- added R12: 3, Resistor_SMD:R_0402_1005Metric, F.Cu at (140.9, 95.5)
- added R13: 10k, Resistor_SMD:R_0402_1005Metric, F.Cu at (140.9, 97.5)
- added R14: 0, Resistor_SMD:R_0402_1005Metric, F.Cu at (140.9, 99.5)
- added R15: 0, Resistor_SMD:R_0402_1005Metric, F.Cu at (140.9, 101.5)
- added REF**: Tag-Connect_TC2050-IDC-FP_2x05_P1.27mm_Vertical, Connector:Tag-Connect_TC2050-IDC-FP_2x05_P1.27mm_Vertical, F.Cu at (128.2, 86.8)
- added U4: Conn, inkbadge:LCSC_1x24-1MP_P0.5mm_Horizontal, F.Cu at (159.6, 101.1)
- C1, C19, C5: footprint Capacitor_SMD:C_0805_2012Metric -> Capacitor_SMD:C_0603_1608Metric
- moved R4 1.02 mm to (115.4, 108.1), turned to 90 degrees
Connections:
- U1 pad 10: /GPIO7 -> unconnected-(U1-GPIO7-Pad10)
- U1 pad 12: /GPIO8 -> unconnected-(U1-GPIO8-Pad12)
- U1 pad 13: /GPIO9 -> unconnected-(U1-GPIO9-Pad13)
- U1 pad 14: /GPIO10 -> unconnected-(U1-GPIO10-Pad14)
- U1 pad 15: /GPIO11 -> unconnected-(U1-GPIO11-Pad15)
- U1 pad 16: /GPIO12 -> unconnected-(U1-GPIO12-Pad16)
- U1 pad 17: /GPIO13 -> unconnected-(U1-GPIO13-Pad17)
- U1 pad 18: /GPIO14 -> unconnected-(U1-GPIO14-Pad18)
- U1 pad 19: /GPIO15 -> unconnected-(U1-GPIO15-Pad19)
- U1 pad 2: /GPIO0 -> unconnected-(U1-GPIO0-Pad2)
- U1 pad 24: /SWCLK -> unconnected-(U1-SWCLK-Pad24)
- U1 pad 25: /SWD -> unconnected-(U1-SWD-Pad25)
- U1 pad 27: /GPIO16 -> unconnected-(U1-GPIO16-Pad27)
- U1 pad 28: /GPIO17 -> unconnected-(U1-GPIO17-Pad28)
- U1 pad 29: /GPIO18 -> unconnected-(U1-GPIO18-Pad29)
- U1 pad 3: /GPIO1 -> unconnected-(U1-GPIO1-Pad3)
- U1 pad 31: /GPIO19 -> unconnected-(U1-GPIO19-Pad31)
- U1 pad 32: /GPIO20 -> unconnected-(U1-GPIO20-Pad32)
- U1 pad 33: /GPIO21 -> unconnected-(U1-GPIO21-Pad33)
- U1 pad 34: /GPIO22 -> unconnected-(U1-GPIO22-Pad34)
- U1 pad 35: /GPIO23 -> unconnected-(U1-GPIO23-Pad35)
- U1 pad 36: /GPIO24 -> unconnected-(U1-GPIO24-Pad36)
- U1 pad 37: /GPIO25 -> unconnected-(U1-GPIO25-Pad37)
- U1 pad 4: /GPIO2 -> unconnected-(U1-GPIO2-Pad4)
- U1 pad 40: /GPIO26_ADC0 -> unconnected-(U1-GPIO26_ADC0-Pad40)
- U1 pad 41: /GPIO27_ADC1 -> unconnected-(U1-GPIO27_ADC1-Pad41)
- U1 pad 42: /GPIO28_ADC2 -> unconnected-(U1-GPIO28_ADC2-Pad42)
- U1 pad 43: /GPIO29_ADC3 -> unconnected-(U1-GPIO29_ADC3-Pad43)
- U1 pad 5: /GPIO3 -> unconnected-(U1-GPIO3-Pad5)
- U1 pad 7: /GPIO4 -> unconnected-(U1-GPIO4-Pad7)
- U1 pad 8: /GPIO5 -> unconnected-(U1-GPIO5-Pad8)
- U1 pad 9: /GPIO6 -> unconnected-(U1-GPIO6-Pad9)
Routing:
- net unconnected-(U1-GPIO15-Pad19): track 0.00 -> 13.3 mm
- net /GPIO15: track 13.3 -> 0.00 mm
- net GND: track 34.1 -> 33.1 mm, vias 26 -> 25
Other:
- board text removed: "DEBUG"
- board text removed: "Minimal Design Example REV3"
- board text removed: "Raspberry Pi RP2350A QFN-60"

Commit message: Progress
Parts:
- removed C28: 1u, Capacitor_SMD:C_0402_1005Metric
- removed C32: 10u, Capacitor_SMD:C_0402_1005Metric
- removed C9: 4.7u, Capacitor_SMD:C_0402_1005Metric
- removed R5: 33, Resistor_SMD:R_0402_1005Metric
- removed REF**: Tag-Connect_TC2050-IDC-FP_2x05_P1.27mm_Vertical, Connector:Tag-Connect_TC2050-IDC-FP_2x05_P1.27mm_Vertical
- added L2: 10uH 1A, Inductor_SMD:L_Ferrocore_DLG-0403, F.Cu at (148.2, 106.0)
- moved J1 65.3 mm to (89.2, 100.2), turned to -90 degrees
- moved U2 40.2 mm to (147.6, 90.0)
- moved R2 39.5 mm to (138.8, 101.7)
- moved R11 39.5 mm to (122.0, 99.0)
- moved R3 39.5 mm to (122.0, 97.0)
- moved C10 39.2 mm to (139.7, 101.7)
- moved C18 39.2 mm to (137.0, 100.5), turned to 180 degrees
- moved C12 39.1 mm to (136.8, 88.5)
- moved C6 39.1 mm to (140.9, 91.3)
- moved C7 39.1 mm to (140.9, 90.4)
- moved L1 39.1 mm to (140.9, 88.7)
- moved R7 39.1 mm to (137.8, 88.5)
- moved R8 39.1 mm to (138.8, 88.5)
- moved U1 39.1 mm to (138.9, 95.9)
- moved C13 39.1 mm to (132.4, 92.5)
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Connections:
- U1 pad 31: unconnected-(U1-GPIO19-Pad31) -> /BUSY
- U1 pad 32: unconnected-(U1-GPIO20-Pad32) -> /~{RES}
- U1 pad 33: unconnected-(U1-GPIO21-Pad33) -> /~{D/C}
- U1 pad 34: unconnected-(U1-GPIO22-Pad34) -> /~{DISCS}
- U1 pad 35: unconnected-(U1-GPIO23-Pad35) -> /SCLK
- U1 pad 36: unconnected-(U1-GPIO24-Pad36) -> /MOSI
- U1 pad 46: /VREG_AVDD -> unconnected-(U1-VREG_AVDD-Pad46)
Routing:
- net GND: track 33.1 -> 6.52 mm, vias 25 -> 9
- net /QSPI_SS: track 21.5 -> 5.40 mm
- net +3V3: track 28.4 -> 14.6 mm
- net /MOSI: track 0.00 -> 13.5 mm
- net /BUSY: track 0.00 -> 13.4 mm
- net /SCLK: track 0.00 -> 13.4 mm
- net /~{RES}: track 0.00 -> 13.3 mm
- net /~{DISCS}: track 0.00 -> 13.3 mm
- net /~{D/C}: track 0.00 -> 13.3 mm
- net unconnected-(U1-GPIO15-Pad19): track 13.3 -> 0.00 mm
- net Net-(D3-A): track 0.00 -> 12.7 mm
- net /QSPI_SD2: track 13.0 -> 0.46 mm
- net /USB_D+: track 12.5 -> 0.58 mm
- net /QSPI_SD1: track 16.7 -> 5.81 mm
- net /VGL: track 0.00 -> 9.26 mm
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- removed copper zone on F.Cu, net VBUS
Other:
- board text removed: "ADC 26-29"
- board text removed: "BOOTSEL"
- board text removed: "Outer Row GND"

Commit message: Journaling
Parts:
- removed J4: USB_C_Receptacle_USB2.0_14P, Connector_USB:USB_C_Receptacle_GCT_USB4105-xx-A_16P_TopMnt_Horizontal
- removed R11, R3: 33, Resistor_SMD:R_0402_1005Metric
- removed R14, R15: 0, Resistor_SMD:R_0402_1005Metric
- removed U3: W25Q128JVS, Package_SO:SOIC-8_5.23x5.23mm_P1.27mm
- added D4: LED, LED_THT:LED_D3.0mm_Horizontal_O1.27mm_Z2.0mm, F.Cu at (52.0, 79.7)
- added D5: LED, LED_THT:LED_D3.0mm_Horizontal_O1.27mm_Z2.0mm, F.Cu at (52.0, 85.7)
- added D6: LED, LED_THT:LED_D3.0mm_Horizontal_O1.27mm_Z2.0mm, F.Cu at (52.0, 91.7)
- added D7: LED, LED_THT:LED_D3.0mm_Horizontal_O1.27mm_Z2.0mm, F.Cu at (52.0, 97.7)
- added J2: Bus_PCI_Express_x4, Connector_PCBEdge:BUS_PCIexpress_x4, F.Cu at (75.0, 79.2)
- added SW3: SW_Push, Button_Switch_SMD:SW_Push_1P1T_NO_CK_KSC6xxJ, F.Cu at (122.5, 120.0)
- added SW4: SW_Push, Button_Switch_SMD:SW_Push_1P1T_NO_CK_KSC6xxJ, F.Cu at (137.5, 120.0)
- added SW5: SW_Push, Button_Switch_SMD:SW_Push_1P1T_NO_CK_KSC6xxJ, F.Cu at (152.5, 120.0)
- added U5: W25Q128JVS, Package_SO:SOIC-8_5.3x5.3mm_P1.27mm, F.Cu at (129.3, 87.7)
- SW1, SW2: footprint Button_Switch_SMD:SW_Push_1P1T_NO_Vertical_Wuerth_434133025816 -> Button_Switch_SMD:SW_SPST_B3U-1000P
- moved C19 50.7 mm to (148.5, 83.8)
- moved C5 43.2 mm to (152.2, 88.4), turned to 90 degrees
- moved R1 34.8 mm to (126.3, 92.0)
- moved R9 34.8 mm to (124.6, 92.0)
- moved C1 34.1 mm to (143.1, 85.9), turned to 90 degrees
- moved R6 31.1 mm to (133.8, 91.5)
- moved C2 27.9 mm to (124.1, 84.3)
- moved J1 25.2 mm to (114.3, 102.1)
- moved R10 20.3 mm to (123.4, 87.5)
- moved SW1 16.1 mm to (129.5, 93.8), turned to 90 degrees
Connections:
- net VBUS renamed +5V
- U1 pad 29: unconnected-(U1-GPIO18-Pad29) -> /BUSY
- U1 pad 31: /BUSY -> /~{RES}
- U1 pad 32: /~{RES} -> /~{D/C}
- U1 pad 33: /~{D/C} -> /~{DISCS}
- U1 pad 34: /~{DISCS} -> /SCLK
- U1 pad 35: /SCLK -> /MOSI
- U1 pad 36: /MOSI -> unconnected-(U1-GPIO24-Pad36)
Routing:
- net /BUSY: track 13.4 -> 15.7 mm, vias 0 -> 2
- net /USB_D+: track 0.58 -> 0.00 mm
- net (no net): vias 0 -> 1
Other:
- board outline added: 82.5 x 57.5 mm

Commit message: Update
Parts:
- removed D5, D6, D7: LED, LED_THT:LED_D3.0mm_Horizontal_O1.27mm_Z2.0mm
- added C28: 10uF, Capacitor_SMD:C_0603_1608Metric, F.Cu at (334.5, 109.0)
- added C9: 10u, Capacitor_SMD:C_0603_1608Metric, F.Cu at (342.4, 111.4)
- added D10: SK6812MINI, LED_SMD:LED_SK6812MINI_PLCC4_3.5x3.5mm_P1.75mm, F.Cu at (322.7, 121.8)
- added D8: SK6812MINI, LED_SMD:LED_SK6812MINI_PLCC4_3.5x3.5mm_P1.75mm, F.Cu at (311.7, 121.8)
- added D9: SK6812MINI, LED_SMD:LED_SK6812MINI_PLCC4_3.5x3.5mm_P1.75mm, F.Cu at (317.2, 121.8)
- added J3: USB_C_Receptacle_USB2.0_14P, Connector_USB:USB_C_Receptacle_GCT_USB4105-xx-A_16P_TopMnt_Horizontal, B.Cu at (350.7, 83.5)
- added J4: Conn_02x06_Odd_Even, Connector_PinSocket_2.54mm:PinSocket_2x06_P2.54mm_Vertical, F.Cu at (310.9, 128.5)
- added J5: Conn_01x02, Connector_PinHeader_2.54mm:PinHeader_1x02_P2.54mm_Vertical, F.Cu at (345.2, 112.5)
- added R3: 5.1k, Resistor_SMD:R_0402_1005Metric, F.Cu at (348.2, 87.2)
- added R5: 5.1k, Resistor_SMD:R_0402_1005Metric, F.Cu at (353.4, 87.3)
- added SW10: SW_Push, Button_Switch_SMD:SW_Push_1P1T_NO_CK_KSC6xxJ, F.Cu at (352.7, 129.8)
- added SW6: SW_Push, Button_Switch_SMD:SW_Push_1P1T_NO_CK_KSC6xxJ, F.Cu at (298.9, 129.8)
- added SW7: SW_Push, Button_Switch_SMD:SW_Push_1P1T_NO_CK_KSC6xxJ, F.Cu at (335.5, 126.1)
- added SW8: SW_Push, Button_Switch_SMD:SW_Push_1P1T_NO_CK_KSC6xxJ, F.Cu at (342.2, 132.8)
- added SW9: SW_Push, Button_Switch_SMD:SW_Push_1P1T_NO_CK_KSC6xxJ, F.Cu at (346.0, 123.1)
- added U3: SRV05-4, Package_TO_SOT_SMD:SOT-23-6, B.Cu at (350.8, 90.4)
- added U6: TP4056-42-ESOP8, inkbadge:SOP-8_3.9x4.9mm_P1.27mm-TP, F.Cu at (338.0, 112.6)
- D4: footprint LED_THT:LED_D3.0mm_Horizontal_O1.27mm_Z2.0mm -> LED_SMD:LED_0603_1608Metric
- J1: moved to B.Cu
- R1: value DNF -> 10k
- R10: value 0 -> 1.5k
- R9: value DNF -> 5k
- moved J2 294.6 mm to (367.1, 117.5), turned to 90 degrees
- moved D4 282.4 mm to (332.6, 110.8), turned to 180 degrees
- moved R9 218.7 mm to (342.2, 113.9)
- moved R10 211.7 mm to (333.6, 112.6), turned to -90 degrees
- moved C2 187.3 mm to (310.9, 96.4), turned to 0 degrees
- moved R1 183.9 mm to (310.0, 101.3), turned to 90 degrees
- moved C1 177.8 mm to (320.7, 93.7), turned to 180 degrees
- moved C13 177.5 mm to (309.6, 102.7)
- moved SW1 177.3 mm to (306.6, 103.3)
- moved C15 177.1 mm to (309.2, 107.0)
- moved C8 177.0 mm to (309.1, 104.6)
- moved C19 176.9 mm to (325.1, 93.7)
- moved C18 176.5 mm to (313.2, 110.8), turned to -90 degrees
- moved C17 176.4 mm to (319.2, 102.4)
- moved C6 176.0 mm to (316.7, 100.9)
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Connections:
- D4 pad 1: unconnected-(D4-K-Pad1) -> Net-(D4-K)
- D4 pad 2: unconnected-(D4-A-Pad2) -> +5V
- J2 pad A10: Net-(J2-+3.3V-PadA10) -> +3V3
- J2 pad A12: Net-(J2-GND-PadA12) -> GND
- J2 pad A15: Net-(J2-GND-PadA12) -> GND
- J2 pad A18: Net-(J2-GND-PadA12) -> GND
- J2 pad A2: Net-(J2-+12V-PadA2) -> +5V
- J2 pad A20: Net-(J2-GND-PadA12) -> GND
- J2 pad A23: Net-(J2-GND-PadA12) -> GND
- J2 pad A24: Net-(J2-GND-PadA12) -> GND
- J2 pad A27: Net-(J2-GND-PadA12) -> GND
- J2 pad A28: Net-(J2-GND-PadA12) -> GND
- J2 pad A3: Net-(J2-+12V-PadA2) -> +5V
- J2 pad A31: Net-(J2-GND-PadA12) -> GND
- J2 pad A4: Net-(J2-GND-PadA12) -> GND
- J2 pad A9: Net-(J2-+3.3V-PadA10) -> +3V3
- J2 pad B1: Net-(J2-+12V-PadA2) -> +5V
- J2 pad B10: unconnected-(J2-3.3Vaux-PadB10) -> +3V3
- J2 pad B13: Net-(J2-GND-PadA12) -> GND
- J2 pad B14: unconnected-(J2-PETp0-PadB14) -> /MISO1
- J2 pad B15: unconnected-(J2-PETn0-PadB15) -> /CS1
- J2 pad B16: Net-(J2-GND-PadA12) -> GND
- J2 pad B18: Net-(J2-GND-PadA12) -> GND
- J2 pad B19: unconnected-(J2-PETp1-PadB19) -> /CLK1
- J2 pad B2: Net-(J2-+12V-PadA2) -> +5V
- J2 pad B20: unconnected-(J2-PETn1-PadB20) -> /MOSI1
- J2 pad B21: Net-(J2-GND-PadA12) -> GND
- J2 pad B22: Net-(J2-GND-PadA12) -> GND
- J2 pad B25: Net-(J2-GND-PadA12) -> GND
- J2 pad B26: Net-(J2-GND-PadA12) -> GND
- J2 pad B29: Net-(J2-GND-PadA12) -> GND
- J2 pad B3: Net-(J2-+12V-PadA2) -> +5V
- J2 pad B32: Net-(J2-GND-PadA12) -> GND
- J2 pad B4: Net-(J2-GND-PadA12) -> GND
- J2 pad B7: Net-(J2-GND-PadA12) -> GND
- J2 pad B8: Net-(J2-+3.3V-PadA10) -> +3V3
- R1 pad 2: /FLASH_SS -> /QSPI_SS
- R10 pad 1: /QSPI_SS -> Net-(D4-K)
- R10 pad 2: /FLASH_SS -> Net-(U6-~{CHRG})
- R7 pad 1: /USB_D+ -> /D+
- R8 pad 1: /USB_D- -> /D-
- R9 pad 1: /GPIO0 -> Net-(U6-PROG)
- R9 pad 2: /FLASH_SS -> GND
- SW3 pad 1: unconnected-(SW3-Pad1) -> /SW1
- SW3 pad 2: unconnected-(SW3-Pad2) -> GND
- SW4 pad 1: unconnected-(SW4-Pad1) -> /SW2
- SW4 pad 2: unconnected-(SW4-Pad2) -> GND
- SW5 pad 1: unconnected-(SW5-Pad1) -> /SW3
- SW5 pad 2: unconnected-(SW5-Pad2) -> GND
- U1 pad 10: unconnected-(U1-GPIO7-Pad10) -> /MOSI
- U1 pad 12: unconnected-(U1-GPIO8-Pad12) -> /SW1
- U1 pad 13: unconnected-(U1-GPIO9-Pad13) -> /SW2
- U1 pad 14: unconnected-(U1-GPIO10-Pad14) -> /SW3
- U1 pad 15: unconnected-(U1-GPIO11-Pad15) -> /SW4
- U1 pad 16: unconnected-(U1-GPIO12-Pad16) -> /SDCS
- U1 pad 17: unconnected-(U1-GPIO13-Pad17) -> /P5
- U1 pad 18: unconnected-(U1-GPIO14-Pad18) -> /P1
- U1 pad 19: unconnected-(U1-GPIO15-Pad19) -> /P6
- U1 pad 27: unconnected-(U1-GPIO16-Pad27) -> /NEOPIXEL_IN
- U1 pad 28: unconnected-(U1-GPIO17-Pad28) -> /P2
- U1 pad 29: /BUSY -> /P3
- U1 pad 3: unconnected-(U1-GPIO1-Pad3) -> /BUSY
- U1 pad 31: /~{RES} -> /P7
- U1 pad 32: /~{D/C} -> /P4
- U1 pad 33: /~{DISCS} -> /P8
- U1 pad 34: /SCLK -> /SW5
- U1 pad 35: /MOSI -> /SW6
- U1 pad 36: unconnected-(U1-GPIO24-Pad36) -> /SW7
- U1 pad 37: unconnected-(U1-GPIO25-Pad37) -> /SW8
- U1 pad 4: unconnected-(U1-GPIO2-Pad4) -> /~{RES}
- U1 pad 40: unconnected-(U1-GPIO26_ADC0-Pad40) -> /CLK1
- U1 pad 41: unconnected-(U1-GPIO27_ADC1-Pad41) -> /MOSI1
- U1 pad 42: unconnected-(U1-GPIO28_ADC2-Pad42) -> /MISO1
- U1 pad 43: unconnected-(U1-GPIO29_ADC3-Pad43) -> /CS1
- U1 pad 5: unconnected-(U1-GPIO3-Pad5) -> /~{D/C}
- U1 pad 7: unconnected-(U1-GPIO4-Pad7) -> /MISO
- U1 pad 8: unconnected-(U1-GPIO5-Pad8) -> /~{DISCS}
- U1 pad 9: unconnected-(U1-GPIO6-Pad9) -> /SCLK
- U5 pad 1: /FLASH_SS -> /QSPI_SS
Routing:
- net +3V3: track 14.6 -> 185.7 mm, vias 0 -> 8
- net +5V: track 0.00 -> 114.7 mm, vias 0 -> 18
- net /SW8: track 0.00 -> 54.4 mm
- net /D+: track 0.00 -> 54.4 mm, vias 0 -> 1
- net /MOSI1: track 0.00 -> 52.7 mm, vias 0 -> 2
- net /CLK1: track 0.00 -> 52.5 mm, vias 0 -> 2
- net /D-: track 0.00 -> 51.2 mm, vias 0 -> 1
- net /CS1: track 0.00 -> 50.0 mm, vias 0 -> 2
- net /MISO1: track 0.00 -> 50.0 mm, vias 0 -> 2
- net /SW6: track 0.00 -> 43.9 mm
- net /SW1: track 0.00 -> 41.0 mm
- net /SW3: track 0.00 -> 40.4 mm
- net /MISO: track 0.00 -> 37.1 mm, vias 0 -> 1
- net /SW7: track 0.00 -> 37.0 mm
- net /SDCS: track 0.00 -> 34.6 mm, vias 0 -> 1
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- added copper zone on B.Cu, net +3V3
- added copper zone on B.Cu, net +5V
- added copper zone on B.Cu, net GND
Other:
- board size 82.5 x 57.5 mm -> 90 x 69 mm

Commit message: Badge like done!
Parts:
- removed J4: Conn_02x06_Odd_Even, Connector_PinSocket_2.54mm:PinSocket_2x06_P2.54mm_Vertical
- removed SW10, SW7, SW8, SW9: SW_Push, Button_Switch_SMD:SW_Push_1P1T_NO_CK_KSC6xxJ
- added C32: 100nF, Capacitor_SMD:C_0402_1005Metric, F.Cu at (133.0, 84.0)
- added C33: 100nF, Capacitor_SMD:C_0402_1005Metric, F.Cu at (129.5, 84.0)
- added C34: 100nF, Capacitor_SMD:C_0402_1005Metric, F.Cu at (76.2, 84.0)
- added C35: 100nF, Capacitor_SMD:C_0402_1005Metric, F.Cu at (80.3, 83.3)
- added C36: 100nF, Capacitor_SMD:C_0402_1005Metric, B.Cu at (105.4, 126.8)
- added C37: 1uF, Capacitor_SMD:C_0402_1005Metric, F.Cu at (72.0, 100.0)
- added C38: 1uF, Capacitor_SMD:C_0402_1005Metric, B.Cu at (80.3, 99.5)
- added C39: 4.7uF, Capacitor_SMD:C_0603_1608Metric, B.Cu at (139.6, 128.2)
- added D11: MBR0530, Diode_SMD:D_SOD-123, B.Cu at (120.7, 125.7)
- added D5: WS2812B-2020, LED_SMD:LED_WS2812B-2020_PLCC4_2.0x2.0mm, F.Cu at (131.5, 82.0)
- added D6: WS2812B-2020, LED_SMD:LED_WS2812B-2020_PLCC4_2.0x2.0mm, F.Cu at (135.0, 82.0)
- added D7: WS2812B-2020, LED_SMD:LED_WS2812B-2020_PLCC4_2.0x2.0mm, F.Cu at (81.5, 82.0)
- added H1: MountingHole, MountingHole:MountingHole_2.2mm_M2_Pad_Via, F.Cu at (67.3, 70.7)
- added H2: MountingHole, MountingHole:MountingHole_2.2mm_M2_Pad_Via, F.Cu at (142.3, 70.7)
- added H3: MountingHole, MountingHole:MountingHole_2.2mm_M2_Pad_Via, F.Cu at (74.0, 140.2)
- added H4: MountingHole, MountingHole:MountingHole_2.2mm_M2_Pad_Via, F.Cu at (134.0, 140.2)
- added JP1: Slice before pluggin into PCIEx4, Jumper:SolderJumper-2_P1.3mm_Bridged_RoundedPad1.0x1.5mm, B.Cu at (145.7, 87.7)
- added Q2: AO3401A, Package_TO_SOT_SMD:SOT-23, B.Cu at (116.4, 125.7)
- added R14: 1.5k, Resistor_SMD:R_0402_1005Metric, B.Cu at (121.2, 127.4)
- C1, C19, C5, C9: value 10u -> 10uF; moved to B.Cu
- C10: value 4.7u -> 4.7uF; moved to B.Cu
- C11, C12, C13, C14, C15, C16, C17, C18, C2, C8: value 100n -> 100nF; moved to B.Cu
- C20, C21, C23, C24, C25, C26, C30, C31: value 1u -> 1uF; moved to B.Cu
- C22: value 1u -> 100nF; moved to B.Cu
- C27, C29: footprint Capacitor_SMD:C_0402_1005Metric -> Capacitor_SMD:C_0603_1608Metric; moved to B.Cu
- C28, D1, D2, D3, D4, J2, L1, L2, Q1, R1, R10, R12, R13, R2, R3, R4, R5, R6, R7, R8, R9, SW1, SW2, U2, U4, U5, U6: moved to B.Cu
- C3, C4: value 15p -> 15pF; moved to B.Cu
- C6, C7: value 4.7u -> 4.7uF; footprint RP2350_60QFN_minimal:C_0402_1005Metric_small_pads -> Capacitor_SMD:C_0402_1005Metric; moved to B.Cu
- D10, D8, D9: value SK6812MINI -> WS2812B-2020; footprint LED_SMD:LED_SK6812MINI_PLCC4_3.5x3.5mm_P1.75mm -> LED_SMD:LED_WS2812B-2020_PLCC4_2.0x2.0mm
- SW3, SW4, SW5, SW6: footprint Button_Switch_SMD:SW_Push_1P1T_NO_CK_KSC6xxJ -> inkbadge:SW_Push_SPST_TSA016
- U1: value ~ -> RP2350A; moved to B.Cu
- Y1: value ABM8-272-T3 -> 12MHz 10pf; footprint Crystal:Crystal_SMD_3225-4Pin_3.2x2.5mm -> Crystal:Crystal_SMD_2520-4Pin_2.5x2.0mm; moved to B.Cu
- moved D10 251.4 mm to (74.5, 82.0), turned to -45 degrees
- moved D9 242.5 mm to (78.0, 82.0), turned to -45 degrees
- moved J5 239.3 mm to (106.0, 119.2), turned to -90 degrees
- moved R4 224.3 mm to (94.7, 96.0), turned to -135 degrees
- moved Y1 222.2 mm to (92.3, 99.6), turned to 45 degrees
- moved SW2 221.9 mm to (96.9, 98.0), turned to -45 degrees
- moved C28 221.1 mm to (114.6, 132.2)
- moved C4 220.9 mm to (95.0, 99.9), turned to 45 degrees
- moved C3 219.9 mm to (93.0, 102.0), turned to -135 degrees
- moved C10 219.2 mm to (96.5, 101.6), turned to 135 degrees
- moved C16 219.1 mm to (99.9, 99.9), turned to 90 degrees
- moved R2 218.9 mm to (95.8, 102.2), turned to 135 degrees
- moved R10 218.5 mm to (115.9, 130.9), turned to 0 degrees
- moved C9 218.4 mm to (125.0, 131.8), turned to 90 degrees
- moved U6 218.2 mm to (120.5, 130.6)
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Connections:
- D10 pad 1: Net-(D10-DOUT) -> unconnected-(D10-DOUT-Pad1)
- D10 pad 3: /NEOPIXEL_IN -> Net-(D10-DIN)
- D8 pad 1: unconnected-(D8-DOUT-Pad1) -> Net-(D5-DIN)
- D8 pad 3: Net-(D8-DIN) -> /NEOPIXEL_IN
- D9 pad 1: Net-(D8-DIN) -> Net-(D10-DIN)
- D9 pad 3: Net-(D10-DOUT) -> Net-(D7-DOUT)
- J1 pad 5: /SCLK -> /CLK
- J2 pad A2: +5V -> Net-(JP1-B)
- J2 pad A3: +5V -> Net-(JP1-B)
- J2 pad B1: +5V -> Net-(JP1-B)
- J2 pad B2: +5V -> Net-(JP1-B)
- J2 pad B3: +5V -> Net-(JP1-B)
- U1 pad 10: /MOSI -> unconnected-(U1-GPIO7-Pad10)
- U1 pad 12: /SW1 -> unconnected-(U1-GPIO8-Pad12)
- U1 pad 13: /SW2 -> /BUSY
- U1 pad 14: /SW3 -> /~{RES}
- U1 pad 15: /SW4 -> /~{D/C}
- U1 pad 16: /SDCS -> /MISO
- U1 pad 17: /P5 -> /~{DISCS}
- U1 pad 18: /P1 -> /CLK
- U1 pad 19: /P6 -> /MOSI
- U1 pad 2: unconnected-(U1-GPIO0-Pad2) -> /SW4
- U1 pad 27: /NEOPIXEL_IN -> /NEOPIXEL_IN2
- U1 pad 28: /P2 -> unconnected-(U1-GPIO17-Pad28)
- U1 pad 29: /P3 -> unconnected-(U1-GPIO18-Pad29)
- U1 pad 3: /BUSY -> /SW3
- U1 pad 31: /P7 -> unconnected-(U1-GPIO19-Pad31)
- U1 pad 32: /P4 -> /MISO1
- U1 pad 33: /P8 -> /CS1
- U1 pad 34: /SW5 -> /CLK1
- U1 pad 35: /SW6 -> /MOSI1
- U1 pad 36: /SW7 -> unconnected-(U1-GPIO24-Pad36)
- U1 pad 37: /SW8 -> unconnected-(U1-GPIO25-Pad37)
- U1 pad 4: /~{RES} -> /SW2
- U1 pad 40: /CLK1 -> /NEOPIXEL_IN
- U1 pad 41: /MOSI1 -> unconnected-(U1-GPIO27_ADC1-Pad41)
- U1 pad 42: /MISO1 -> unconnected-(U1-GPIO28_ADC2-Pad42)
- U1 pad 43: /CS1 -> unconnected-(U1-GPIO29_ADC3-Pad43)
- U1 pad 5: /~{D/C} -> unconnected-(U1-GPIO3-Pad5)
- U1 pad 7: /MISO -> /SW1
- U1 pad 8: /~{DISCS} -> /SDCS
- U1 pad 9: /SCLK -> unconnected-(U1-GPIO6-Pad9)
- U4 pad 13: /SCLK -> /CLK
- U4 pad 19: unconnected-(U4-VPP-Pad19) -> Net-(U4-VPP)
Routing:
- net /CLK: track 0.00 -> 63.0 mm, vias 0 -> 2
- net /SW8: track 54.4 -> 0.00 mm
- net /SW6: track 43.9 -> 0.00 mm
- net /SCLK: track 42.0 -> 0.00 mm, vias 1 -> 0
- net /SW7: track 37.0 -> 0.00 mm
- net /P8: track 32.0 -> 0.00 mm
- net /P7: track 31.5 -> 0.00 mm
- net /P2: track 30.7 -> 0.00 mm
- net /P3: track 29.6 -> 0.00 mm
- net /SW5: track 29.3 -> 0.00 mm
- net /P6: track 28.8 -> 0.00 mm
- net /P5: track 28.5 -> 0.00 mm
- net /P4: track 28.3 -> 0.00 mm
- net /NEOPIXEL_IN2: track 0.00 -> 26.6 mm, vias 0 -> 1
- net /P1: track 25.3 -> 0.00 mm
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- added copper zone on B.Cu, net +1V1
- added copper zone on B.Cu, net /VREG_LX
- added copper zone on B.Cu, net Net-(JP1-B)
- removed copper zone on F.Cu, net +1V1
- removed copper zone on F.Cu, net +3V3
- removed copper zone on F.Cu, net /VREG_LX
Other:
- board size 90 x 69 mm -> 88.9 x 91.3 mm
- board text added: "BOOT"

Commit message: Finish programmer
Parts:
- added JP2: SolderJumper_2_Open, Jumper:SolderJumper-2_P1.3mm_Open_RoundedPad1.0x1.5mm, B.Cu at (146.2, 95.3)
- moved C6 4.78 mm to (109.5, 108.0)
- moved C7 4.78 mm to (110.1, 108.7)
- moved U2 4.78 mm to (115.6, 104.7)
- moved U5 4.78 mm to (104.7, 117.8)
- moved C1 4.78 mm to (117.4, 110.2)
- moved C10 4.78 mm to (101.3, 101.6)
- moved C11 4.78 mm to (109.3, 102.1)
- moved C12 4.78 mm to (108.2, 112.6)
- moved C13 4.78 mm to (103.2, 111.7)
- moved C14 4.78 mm to (108.7, 101.5)
- moved C15 4.78 mm to (99.9, 108.9)
- moved C16 4.78 mm to (104.6, 99.9)
- moved C17 4.78 mm to (110.2, 105.2)
- moved C18 4.78 mm to (100.1, 103.5)
- moved C19 4.78 mm to (120.5, 107.1)
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Connections:
- J2 pad A10: +3V3 -> Net-(J2-3.3Vaux)
- J2 pad A5: unconnected-(J2-JTAG2-PadA5) -> /CLK1
- J2 pad A6: unconnected-(J2-JTAG3-PadA6) -> /MOSI1
- J2 pad A7: unconnected-(J2-JTAG4-PadA7) -> /MISO1
- J2 pad A8: unconnected-(J2-JTAG5-PadA8) -> /CS1
- J2 pad A9: +3V3 -> Net-(J2-3.3Vaux)
- J2 pad B10: +3V3 -> Net-(J2-3.3Vaux)
- J2 pad B14: /MISO1 -> unconnected-(J2-PETp0-PadB14)
- J2 pad B15: /CS1 -> unconnected-(J2-PETn0-PadB15)
- J2 pad B19: /CLK1 -> unconnected-(J2-PETp1-PadB19)
- J2 pad B20: /MOSI1 -> unconnected-(J2-PETn1-PadB20)
- J2 pad B5: unconnected-(J2-SMCLK-PadB5) -> /I2C_CLK
- J2 pad B6: unconnected-(J2-SMDAT-PadB6) -> /I2C_DATA
- J2 pad B8: +3V3 -> Net-(J2-3.3Vaux)
- U1 pad 42: unconnected-(U1-GPIO28_ADC2-Pad42) -> /I2C_DATA
- U1 pad 43: unconnected-(U1-GPIO29_ADC3-Pad43) -> /I2C_CLK
Routing:
- net /I2C_CLK: track 0.00 -> 52.4 mm, vias 0 -> 2
- net /I2C_DATA: track 0.00 -> 50.9 mm, vias 0 -> 2
- net Net-(J2-3.3Vaux): track 0.00 -> 20.6 mm, vias 0 -> 2
- net +3V3: track 161.9 -> 149.2 mm, vias 16 -> 15
- net /CLK: track 63.0 -> 68.1 mm
- net /MOSI1: track 56.7 -> 51.9 mm, vias 0 -> 1
- net /~{RES}: track 25.8 -> 30.6 mm
- net /MISO: track 41.5 -> 46.3 mm
- net /~{D/C}: track 25.4 -> 30.2 mm
- net /~{DISCS}: track 25.7 -> 30.5 mm
- net /BUSY: track 26.3 -> 31.1 mm
- net /MOSI: track 61.9 -> 66.7 mm
- net /D-: track 48.0 -> 43.2 mm
- net /D+: track 47.8 -> 43.0 mm
- net /CLK1: track 57.1 -> 52.5 mm, vias 0 -> 1
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