File: inkbadge/inkbadge.kicad_pcb (KiCad board)
At the start: 2 copper layers, 88.9 x 91.3 mm, 90 parts, among them J1 Micro_SD_Card, J2 Bus_PCI_Express_x4, J3 USB_C_Receptacle_USB2.0_14P, J5 Conn_01x02, Q1 Si1308EDL, Q2 AO3401A, SW1 SW_Push, SW2 SW_Push, SW3 SW_Push, SW4 SW_Push, SW5 SW_Push, SW6 SW_Push, U1 RP2350A, U2 NCP1117-3.3_SOT223, U3 SRV05-4, U4 Conn, U5 W25Q128JVS, U6 TP4056-42-ESOP8, Y1 12MHz 10pf

Commit message: PUSH
Parts:
- removed Q1: Si1308EDL, Package_TO_SOT_SMD:SOT-323_SC-70
- added C40: 4.7uF, Capacitor_SMD:C_0402_1005Metric, B.Cu at (110.9, 106.4)
- added G***: LOGO, LOGO, B.Cu at (126.2, 68.5)
- added G***: LOGO, LOGO, B.Cu at (121.8, 137.6)
- added G***: LOGO, LOGO, B.Cu at (122.1, 137.5)
- added G***: LOGO, LOGO, B.Cu at (109.2, 105.2)
- added JP3: SolderJumper_2_Open, Jumper:SolderJumper-2_P1.3mm_Open_RoundedPad1.0x1.5mm, B.Cu at (125.4, 123.1)
- added Q3: IRLML2060, Package_TO_SOT_SMD:SOT-23, B.Cu at (75.3, 110.8)
- added R11: 470, Resistor_SMD:R_0402_1005Metric, F.Cu at (124.5, 84.0)
- added R15: 470, Resistor_SMD:R_0402_1005Metric, F.Cu at (99.0, 96.8)
- added R16: 33, Resistor_SMD:R_0402_1005Metric, B.Cu at (111.6, 107.8)
- L2: footprint Inductor_SMD:L_Ferrocore_DLG-0403 -> Inductor_SMD:L_APV_ANR4018
- R12: value 3 -> 0.47
- R9: value 5k -> 5.1k
- SW1, SW2: footprint Button_Switch_SMD:SW_SPST_B3U-1000P -> inkbadge:SW_Push_SPST_TSA016
- Y1: footprint Crystal:Crystal_SMD_2520-4Pin_2.5x2.0mm -> Crystal:Crystal_SMD_3225-4Pin_3.2x2.5mm
- moved C39 23.3 mm to (122.5, 112.3)
- moved C38 8.18 mm to (83.3, 107.1), turned to 0 degrees
- moved R4 6.59 mm to (105.5, 98.8), turned to -45 degrees
- moved R13 3.47 mm to (74.2, 112.7), turned to 90 degrees
- moved C29 2.30 mm to (83.2, 110.7)
- moved SW1 2.29 mm to (99.6, 115.5), turned to -135 degrees
- moved C22 1.02 mm to (74.5, 102.1)
- moved C24 1.02 mm to (74.8, 98.7)
- moved C27 1.02 mm to (78.6, 109.3)
- moved C31 1.02 mm to (76.3, 101.0)
- moved D2 1.02 mm to (77.8, 107.4)
- moved C20 1.02 mm to (74.5, 107.2)
- moved C21 1.02 mm to (74.5, 101.2)
- moved C23 1.02 mm to (74.5, 100.2)
- moved C25 1.02 mm to (74.5, 97.2)
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Connections:
- C9 pad 1: +5V -> VBUS
- D11 pad 1: Net-(D11-K) -> +5V
- D11 pad 2: +5V -> VBUS
- D4 pad 2: +5V -> VBUS
- D7 pad 3: /NEOPIXEL_IN2 -> Net-(D7-DIN)
- D8 pad 3: /NEOPIXEL_IN -> Net-(D8-DIN)
- H1 pad 1: (no net) -> GND
- H2 pad 1: (no net) -> GND
- H3 pad 1: (no net) -> GND
- H4 pad 1: (no net) -> GND
- J3 pad A4: +5V -> VBUS
- J3 pad A9: +5V -> VBUS
- J3 pad B4: +5V -> VBUS
- J3 pad B9: +5V -> VBUS
- Q2 pad 1: +5V -> VBUS
- Q2 pad 2: Net-(D11-K) -> +5V
- R14 pad 1: +5V -> VBUS
- U1 pad 32: /MISO1 -> /MOSI1
- U1 pad 35: /MOSI1 -> /MISO1
- U1 pad 40: /NEOPIXEL_IN -> unconnected-(U1-GPIO26_ADC0-Pad40)
- U1 pad 41: unconnected-(U1-GPIO27_ADC1-Pad41) -> /NEOPIXEL_IN
- U1 pad 46: unconnected-(U1-VREG_AVDD-Pad46) -> Net-(U1-VREG_AVDD)
- U3 pad 5: +5V -> VBUS
- U6 pad 4: +5V -> VBUS
- U6 pad 8: +5V -> VBUS
Routing:
- net VBUS: track 0.00 -> 26.3 mm, vias 0 -> 7
- net /NEOPIXEL_IN2: track 31.0 -> 7.28 mm
- net Net-(D7-DIN): track 0.00 -> 22.6 mm
- net +3V3: track 149.2 -> 129.2 mm, vias 15 -> 13
- net +5V: track 122.2 -> 135.6 mm, vias 16 -> 8
- net /MISO: track 46.3 -> 34.9 mm
- net /SDCS: track 34.4 -> 25.2 mm
- net /CLK: track 68.1 -> 59.9 mm
- net /MOSI: track 66.7 -> 59.0 mm
- net /NEOPIXEL_IN: track 32.4 -> 27.5 mm
- net /SW3: track 20.5 -> 25.4 mm
- net /~{USB_BOOT}: track 2.04 -> 6.80 mm
- net /RUN: track 3.61 -> 7.76 mm
- net Net-(D11-K): track 4.02 -> 0.00 mm
- net Net-(R4-Pad1): track 1.41 -> 5.27 mm
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- added copper zone on B.Cu, net VBUS
Other:
- board text added: "@ GitHub HQ San Francisco"
- board text added: "July 11 - 14"
