File: inkbadge/inkbadge.kicad_pcb (KiCad board)
At the start: 2 copper layers, 88.9 x 91.3 mm, 99 parts, among them J1 Micro_SD_Card, J2 Bus_PCI_Express_x4, J3 USB_C_Receptacle_USB2.0_14P, J5 Conn_01x02, Q2 AO3401A, Q3 IRLML2060, SW1 SW_Push, SW2 SW_Push, SW3 SW_Push, SW4 SW_Push, SW5 SW_Push, SW6 SW_Push, U1 RP2350A, U2 NCP1117-3.3_SOT223, U3 SRV05-4, U4 Conn, U5 W25Q128JVS, U6 TP4056-42-ESOP8, Y1 12MHz 10pf

Commit message: FIRMWARE IDKFHRGVKQHBJ
Parts:
- removed the G*** at (109.2, 105.2)
