File: inkbadge/inkbadge.kicad_sch (KiCad schematic)
At the start: 38 parts, among them J4 USB_C_Receptacle_USB2.0_14P, SW1 SW_Push, SW2 SW_Push, U2 NCP1117-3.3_SOT223, U3 W25Q128JVS, Y1 ABM8-272-T3

Commit message: Progress
Parts:
- added C20, C28, C30: 1u, Capacitor_SMD:C_0402_1005Metric, symbol Device:C_Small
- added C21, C22, C23, C24, C25, C26, C31: 1u, Capacitor_SMD:C_0402_1005Metric, symbol Device:C
- added C27, C29: 4.7uF, Capacitor_SMD:C_0402_1005Metric, symbol Device:C
- added C32: 10u, Capacitor_SMD:C_0402_1005Metric, symbol Device:C_Small
- added D1, D2, D3: MBR0530, Diode_SMD:D_SOD-123, symbol Diode:MBR0530
- added J1: Micro_SD_Card, inkbadge:SDCardlcsc, symbol Connector:Micro_SD_Card_Det1
- added L2: 10uH 1A, symbol Device:L
- added Q1: Si1308EDL, Package_TO_SOT_SMD:SOT-323_SC-70, symbol Transistor_FET:Si1308EDL
- added R12: 3, Resistor_SMD:R_0402_1005Metric, symbol Device:R
- added R13: 10k, Resistor_SMD:R_0402_1005Metric, symbol Device:R
- added R14, R15: 0, Resistor_SMD:R_0402_1005Metric, symbol Device:R
- added U4: Conn, inkbadge:LCSC_1x24-1MP_P0.5mm_Horizontal, symbol inkbadge:EINK-2.9inch
- C1, C19, C5: footprint Capacitor_SMD:C_0805_2012Metric -> Capacitor_SMD:C_0603_1608Metric
Connections:
- net +3V3: now also C22.1, C28.1, C29.1, C32.1, J1.4 (VDD), L2.1, R14.2, U4.15 (VDDIO), U4.16 (VCI)
- net GND: now also C20.2, C21.2, C22.2, C23.2, C24.2, C25.2, C26.2, C28.2, C29.2, C30.2, C31.2, C32.2, D2.1 (K), J1.10 (SHIELD), J1.6 (VSS), R12.2, R13.1, R15.1, U4.17 (VSS), U4.8 (BS1), U4.MP (SHIELD)
- net GPIO0: no longer U1.2 (GPIO0)
- net GPIO1: no longer names the net of U1.3 (GPIO1)
- net GPIO10: no longer names the net of U1.14 (GPIO10)
- net GPIO11: no longer names the net of U1.15 (GPIO11)
- net GPIO12: no longer names the net of U1.16 (GPIO12)
- net GPIO13: no longer names the net of U1.17 (GPIO13)
- net GPIO14: no longer names the net of U1.18 (GPIO14)
- net GPIO15: no longer names the net of U1.19 (GPIO15)
- net GPIO16: no longer names the net of U1.27 (GPIO16)
- net GPIO17: no longer names the net of U1.28 (GPIO17)
- net GPIO18: no longer names the net of U1.29 (GPIO18)
- net GPIO19: no longer names the net of U1.31 (GPIO19)
- net GPIO2: no longer names the net of U1.4 (GPIO2)
- net GPIO20: no longer names the net of U1.32 (GPIO20)
- net GPIO21: no longer names the net of U1.33 (GPIO21)
- net GPIO22: no longer names the net of U1.34 (GPIO22)
- net GPIO23: no longer names the net of U1.35 (GPIO23)
- net GPIO24: no longer names the net of U1.36 (GPIO24)
- net GPIO25: no longer names the net of U1.37 (GPIO25)
- net GPIO26_ADC0: no longer names the net of U1.40 (GPIO26_ADC0)
- net GPIO27_ADC1: no longer names the net of U1.41 (GPIO27_ADC1)
- net GPIO28_ADC2: no longer names the net of U1.42 (GPIO28_ADC2)
- net GPIO29_ADC3: no longer names the net of U1.43 (GPIO29_ADC3)
- net GPIO3: no longer names the net of U1.5 (GPIO3)
- net GPIO4: no longer names the net of U1.7 (GPIO4)
- net GPIO5: no longer names the net of U1.8 (GPIO5)
- net GPIO6: no longer names the net of U1.9 (GPIO6)
- net GPIO7: no longer names the net of U1.10 (GPIO7)
- net GPIO8: no longer names the net of U1.12 (GPIO8)
- net GPIO9: no longer names the net of U1.13 (GPIO9)
- net SWCLK: no longer names the net of U1.24 (SWCLK)
- net SWD: no longer names the net of U1.25 (SWD)
- new net: C27.2, D3.2 (A), L2.2, Q1.3 (D)
- new net: C20.1, U4.4 (VGL/NC)
- new net: C21.1, U4.18 (VDD)
- new net: C23.1, U4.20 (VSH1)
- new net: C24.1, U4.22 (VSL)
- new net: C25.1, U4.24 (VCOM)
- new net: C30.1, U4.5 (VSH2)
- new net: C27.1, D1.1 (K), D2.2 (A)
- new net BUSY: U4.9 (BUSY)
- new net DET: J1.9 (DET)
- new net GDR: Q1.1 (G), R13.2, U4.2 (GDR)
- new net MISO: J1.7 (DAT0)
- new net MOSI: J1.3 (CMD), U4.14 (SDA)
- new net RESE: Q1.2 (S), R12.1, U4.3 (RESE)
- new net SCLK: J1.5 (CLK), U4.13 (SCL)
- new net SDCS: J1.2 (DAT3/CD)
- new net VGH: C31.1, D3.1 (K), U4.21 (VGH)
- new net VGL: C26.1, D1.2 (A), U4.23 (VGL)
- new net ~{DISCS}: U4.12 (~{CS})
- new net ~{D/C}: U4.11 (~{D/C})
- new net ~{RES}: R14.1, R15.2, U4.10 (~{RST})
- no-connect marks 0 -> 5
Other:
- note added: "C20 & C30 can be removed"
- note added: "VGL and VGH caps on conn side"
- note removed: "IOs"
- moved on the sheet: C19

Commit message: Progress
Parts:
- removed C28: 1u, Capacitor_SMD:C_0402_1005Metric, symbol Device:C_Small
- removed C32: 10u, Capacitor_SMD:C_0402_1005Metric, symbol Device:C_Small
- removed C9: 4.7u, Capacitor_SMD:C_0402_1005Metric, symbol Device:C
- removed R5: 33, Resistor_SMD:R_0402_1005Metric, symbol Device:R
- L2: footprint (none) -> Inductor_SMD:L_Ferrocore_DLG-0403; LCSC Part # (none) -> C2929419
Connections:
- net BUSY: now also U1.31 (GPIO19)
- net MOSI: now also U1.36 (GPIO24)
- net SCLK: now also U1.35 (GPIO23)
- net ~{DISCS}: now also U1.34 (GPIO22)
- net ~{D/C}: now also U1.33 (GPIO21)
- net ~{RES}: now also U1.32 (GPIO20)
- net VREG_AVDD: no longer names the net of U1.46 (VREG_AVDD)

Commit message: Journaling
Parts:
- removed J4: USB_C_Receptacle_USB2.0_14P, Connector_USB:USB_C_Receptacle_GCT_USB4105-xx-A_16P_TopMnt_Horizontal, symbol Connector:USB_C_Receptacle_USB2.0_14P
- removed R11, R3: 33, Resistor_SMD:R_0402_1005Metric, symbol Device:R
- removed R14, R15: 0, Resistor_SMD:R_0402_1005Metric, symbol Device:R
- removed U3: W25Q128JVS, Package_SO:SOIC-8_5.23x5.23mm_P1.27mm, symbol Memory_Flash:W25Q128JVS
- added D4, D5, D6, D7: LED, LED_THT:LED_D3.0mm_Horizontal_O1.27mm_Z2.0mm, symbol Device:LED
- added J2: Bus_PCI_Express_x4, Connector_PCBEdge:BUS_PCIexpress_x4, symbol Connector:Bus_PCI_Express_x4
- added SW3, SW4, SW5: SW_Push, Button_Switch_SMD:SW_Push_1P1T_NO_CK_KSC6xxJ, symbol Switch:SW_Push
- added U5: W25Q128JVS, Package_SO:SOIC-8_5.3x5.3mm_P1.27mm, symbol Memory_Flash:W25Q128JVS
- SW1, SW2: footprint Button_Switch_SMD:SW_Push_1P1T_NO_Vertical_Wuerth_434133025816 -> Button_Switch_SMD:SW_SPST_B3U-1000P
Connections:
- net +3V3: now also U5.8 (VCC)
- net BUSY: now also U1.29 (GPIO18); no longer U1.31 (GPIO19)
- net FLASH_SS: now also U5.1 (~{CS})
- net GND: now also U5.4 (GND)
- net MOSI: now also U1.35 (GPIO23); no longer U1.36 (GPIO24)
- net QSPI_SCLK: now also U5.6 (CLK)
- net QSPI_SD0: now also U5.5 (DI/IO_{0})
- net QSPI_SD1: now also U5.2 (DO/IO_{1})
- net QSPI_SD2: now also U5.3 (~{WP}/IO_{2})
- net QSPI_SD3: now also U5.7 (~{HOLD}/~{RESET}/IO_{3})
- net SCLK: now also U1.34 (GPIO22); no longer U1.35 (GPIO23)
- net ~{DISCS}: now also U1.33 (GPIO21); no longer U1.34 (GPIO22)
- net ~{D/C}: now also U1.32 (GPIO20); no longer U1.33 (GPIO21)
- net ~{RES}: now also U1.31 (GPIO19); no longer U1.32 (GPIO20)
- net VBUS renamed +5V
- new net: J2.A10 (+3.3V), J2.A9 (+3.3V), J2.B8 (+3.3V)
- new net: J2.A12 (GND), J2.A15 (GND), J2.A18 (GND), J2.A20 (GND), J2.A23 (GND), J2.A24 (GND), J2.A27 (GND), J2.A28 (GND), J2.A31 (GND), J2.A4 (GND), J2.B13 (GND), J2.B16 (GND), J2.B18 (GND), J2.B21 (GND), J2.B22 (GND), J2.B25 (GND), J2.B26 (GND), J2.B29 (GND), J2.B32 (GND), J2.B4 (GND), J2.B7 (GND)
- new net: J2.A2 (+12V), J2.A3 (+12V), J2.B1 (+12V), J2.B2 (+12V), J2.B3 (+12V)
Other:
- note added: "SPI0"
- note added: "fake pci"
- moved on the sheet: C2, R1, R10, R9

Commit message: Update
Parts:
- removed D5, D6, D7: LED, LED_THT:LED_D3.0mm_Horizontal_O1.27mm_Z2.0mm, symbol Device:LED
- added C28: 10uF, Capacitor_SMD:C_0603_1608Metric, symbol Device:C_Small
- added C9: 10u, Capacitor_SMD:C_0603_1608Metric, symbol Device:C
- added D10, D8, D9: SK6812MINI, LED_SMD:LED_SK6812MINI_PLCC4_3.5x3.5mm_P1.75mm, symbol LED:SK6812MINI
- added J3: USB_C_Receptacle_USB2.0_14P, Connector_USB:USB_C_Receptacle_GCT_USB4105-xx-A_16P_TopMnt_Horizontal, symbol Connector:USB_C_Receptacle_USB2.0_14P
- added J4: Conn_02x06_Odd_Even, Connector_PinSocket_2.54mm:PinSocket_2x06_P2.54mm_Vertical, symbol Connector_Generic:Conn_02x06_Odd_Even
- added J5: Conn_01x02, Connector_PinHeader_2.54mm:PinHeader_1x02_P2.54mm_Vertical, symbol Connector_Generic:Conn_01x02
- added R3, R5: 5.1k, Resistor_SMD:R_0402_1005Metric, symbol Device:R
- added SW10, SW6, SW7, SW8, SW9: SW_Push, Button_Switch_SMD:SW_Push_1P1T_NO_CK_KSC6xxJ, symbol Switch:SW_Push
- added U3: SRV05-4, Package_TO_SOT_SMD:SOT-23-6, symbol Power_Protection:SRV05-4
- added U6: TP4056-42-ESOP8, inkbadge:SOP-8_3.9x4.9mm_P1.27mm-TP, symbol Battery_Management:TP4056-42-ESOP8
- D4: footprint LED_THT:LED_D3.0mm_Horizontal_O1.27mm_Z2.0mm -> LED_SMD:LED_0603_1608Metric
- R1: value DNF -> 10k
- R10: value 0 -> 1.5k
- R9: value DNF -> 5k
Connections:
- net +3V3: now also J2.A10 (+3.3V), J2.A9 (+3.3V), J2.B10 (3.3Vaux), J2.B8 (+3.3V), J4.1 (Pin_1), J4.12 (Pin_12)
- net +5V: now also D4.2 (A), J2.A2 (+12V), J2.A3 (+12V), J2.B1 (+12V), J2.B2 (+12V), J2.B3 (+12V), C9.1, D10.4 (VDD), D8.4 (VDD), D9.4 (VDD), J3.A4 (VBUS), J3.A9 (VBUS), J3.B4 (VBUS), J3.B9 (VBUS), U3.5 (VP), U6.4 (V_{CC}), U6.8 (CE)
- net BUSY: now also U1.3 (GPIO1); no longer U1.29 (GPIO18)
- net GND: now also J2.A12 (GND), J2.A15 (GND), J2.A18 (GND), J2.A20 (GND), J2.A23 (GND), J2.A24 (GND), J2.A27 (GND), J2.A28 (GND), J2.A31 (GND), J2.A4 (GND), J2.B13 (GND), J2.B16 (GND), J2.B18 (GND), J2.B21 (GND), J2.B22 (GND), J2.B25 (GND), J2.B26 (GND), J2.B29 (GND), J2.B32 (GND), J2.B4 (GND), J2.B7 (GND), R9.2, SW3.2, SW4.2, SW5.2, C28.2, C9.2, D10.2 (VSS), D8.2 (VSS), D9.2 (VSS), J3.A1 (GND), J3.A12 (GND), J3.B1 (GND), J3.B12 (GND), J3.S1 (SHIELD), J4.11 (Pin_11), J4.2 (Pin_2), J5.1 (Pin_1), R3.2, R5.2, SW10.2, SW6.2, SW7.2, SW8.2, SW9.2, U3.2 (VN), U6.1 (TEMP), U6.3 (GND), U6.9 (EPAD)
- net MISO: now also U1.7 (GPIO4)
- net MOSI: now also U1.10 (GPIO7); no longer U1.35 (GPIO23)
- net QSPI_SS: now also R1.2, U5.1 (~{CS}); no longer R10.1
- net SCLK: now also U1.9 (GPIO6); no longer U1.34 (GPIO22)
- net SDCS: now also U1.16 (GPIO12)
- net ~{DISCS}: now also U1.8 (GPIO5); no longer U1.33 (GPIO21)
- net ~{D/C}: now also U1.5 (GPIO3); no longer U1.32 (GPIO20)
- net ~{RES}: now also U1.4 (GPIO2); no longer U1.31 (GPIO19)
- net MISO1: now reaches J2.B14 (PETp0)
- net MISO1: now also U1.42 (GPIO28_ADC2)
- net CS1: now reaches J2.B15 (PETn0)
- net CS1: now also U1.43 (GPIO29_ADC3)
- net CLK1: now reaches J2.B19 (PETp1)
- net CLK1: now also U1.40 (GPIO26_ADC0)
- net MOSI1: now reaches J2.B20 (PETn1)
- net MOSI1: now also U1.41 (GPIO27_ADC1)
- net SW3: now reaches SW5.1
- net SW3: now also U1.14 (GPIO10)
- net at D4.1 (K): now also R10.1
- net SW1: now reaches SW3.1
- net SW1: now also U1.12 (GPIO8)
- net SW2: now reaches SW4.1
- net SW2: now also U1.13 (GPIO9)
- net SW4: now reaches U1.15 (GPIO11)
- net SW4: now also SW6.1
- net P5: now reaches U1.17 (GPIO13)
- net P5: now also J4.4 (Pin_4)
- net P1: now reaches U1.18 (GPIO14)
- net P1: now also J4.3 (Pin_3)
- net P6: now reaches U1.19 (GPIO15)
- net P6: now also J4.6 (Pin_6)
- net NEOPIXEL_IN: now reaches U1.27 (GPIO16)
- net NEOPIXEL_IN: now also D10.3 (DIN)
- net P2: now reaches U1.28 (GPIO17)
- net P2: now also J4.5 (Pin_5)
- net SW7: now reaches U1.36 (GPIO24)
- net SW7: now also SW9.1
- net SW8: now reaches U1.37 (GPIO25)
- net SW8: now also SW10.1
- removed net FLASH_SS: R1.2, R10.2, R9.2, U5.1 (~{CS})
- net GPIO0: no longer names the net of R9.1
- net GPIO0: now also U6.2 (PROG)
- net USB_D+ renamed D+
- net D+: now also J3.A6 (D+), J3.B6 (D+), U3.3 (IO2), U3.4 (IO3)
- net USB_D- renamed D-
- net D-: now also J3.A7 (D-), J3.B7 (D-), U3.1 (IO1), U3.6 (IO4)
- new net: R10.2, U6.7 (~{CHRG})
- new net: D8.3 (DIN), D9.1 (DOUT)
- new net: J3.B5 (CC2), R5.1
- new net: D10.1 (DOUT), D9.3 (DIN)
- new net: J3.A5 (CC1), R3.1
- new net +BATT: C28.1, J5.2 (Pin_2), U6.5 (BAT)
- new net P3: J4.7 (Pin_7), U1.29 (GPIO18)
- new net P4: J4.9 (Pin_9), U1.32 (GPIO20)
- new net P7: J4.8 (Pin_8), U1.31 (GPIO19)
- new net P8: J4.10 (Pin_10), U1.33 (GPIO21)
- new net SW5: SW7.1, U1.34 (GPIO22)
- new net SW6: SW8.1, U1.35 (GPIO23)
- no-connect marks 5 -> 9
Other:
- note added: "TODO: Ideal diode if there is the budget"
- note removed: "Make sure R7 and R8 are close to RP2350"
- note removed: "SPI0"
- note removed: "fake pci"
- moved on the sheet: C20, C21, C22, C23, C24, C25, C26, C27, C29, C30, C31, D1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

Commit message: Badge like done!
Parts:
- removed D10, D8, D9: SK6812MINI, LED_SMD:LED_SK6812MINI_PLCC4_3.5x3.5mm_P1.75mm, symbol LED:SK6812MINI
- removed J4: Conn_02x06_Odd_Even, Connector_PinSocket_2.54mm:PinSocket_2x06_P2.54mm_Vertical, symbol Connector_Generic:Conn_02x06_Odd_Even
- removed SW10, SW7, SW8, SW9: SW_Push, Button_Switch_SMD:SW_Push_1P1T_NO_CK_KSC6xxJ, symbol Switch:SW_Push
- added C32, C33, C34, C35: 100nF, Capacitor_SMD:C_0402_1005Metric, symbol Device:C
- added C36: 100nF, Capacitor_SMD:C_0402_1005Metric, symbol Device:C_Small
- added C37, C38: 1uF, Capacitor_SMD:C_0402_1005Metric, symbol Device:C
- added C39: 4.7uF, Capacitor_SMD:C_0603_1608Metric, symbol Device:C
- added D10, D5, D6, D7, D8, D9: WS2812B-2020, LED_SMD:LED_WS2812B-2020_PLCC4_2.0x2.0mm, symbol LED:WS2812B-2020
- added D11: MBR0530, Diode_SMD:D_SOD-123, symbol Diode:MBR0530
- added H1, H2, H3, H4: MountingHole, MountingHole:MountingHole_2.2mm_M2_Pad_Via, symbol Mechanical:MountingHole
- added JP1: Slice before pluggin into PCIEx4, Jumper:SolderJumper-2_P1.3mm_Bridged_RoundedPad1.0x1.5mm, symbol Jumper:SolderJumper_2_Bridged
- added Q2: AO3401A, Package_TO_SOT_SMD:SOT-23, symbol Transistor_FET:AO3401A
- added R14: 1.5k, Resistor_SMD:R_0402_1005Metric, symbol Device:R
- C1, C19, C5: value 10u -> 10uF; symbol Device:C -> Device:C_Small
- C10: value 4.7u -> 4.7uF
- C11, C12, C13, C14, C15, C16, C17, C18, C2, C8: value 100n -> 100nF
- C20, C21, C23, C24, C25, C26, C30, C31: value 1u -> 1uF
- C22: value 1u -> 100nF
- C27, C29: footprint Capacitor_SMD:C_0402_1005Metric -> Capacitor_SMD:C_0603_1608Metric
- C3, C4: value 15p -> 15pF
- C6, C7: value 4.7u -> 4.7uF; footprint RP2350_60QFN_minimal:C_0402_1005Metric_small_pads -> Capacitor_SMD:C_0402_1005Metric
- C9: value 10u -> 10uF
- SW3, SW4, SW5, SW6: footprint Button_Switch_SMD:SW_Push_1P1T_NO_CK_KSC6xxJ -> inkbadge:SW_Push_SPST_TSA016; LCSC Part # (none) -> C2888430
- U1: value ~ -> RP2350A
- Y1: value ABM8-272-T3 -> 12MHz 10pf; footprint Crystal:Crystal_SMD_3225-4Pin_3.2x2.5mm -> Crystal:Crystal_SMD_2520-4Pin_2.5x2.0mm; LCSC Part # (none) -> C7301971
Connections:
- net P4 is gone; now on net MISO1: U1.32 (GPIO20)
- net P5 is gone; now on net ~{DISCS}: U1.17 (GPIO13)
- net P6 is gone; now on net MOSI: U1.19 (GPIO15)
- net P8 is gone; now on net CS1: U1.33 (GPIO21)
- net SW5 is gone; now on net CLK1: U1.34 (GPIO22)
- net SW6 is gone; now on net MOSI1: U1.35 (GPIO23)
- net +3V3: now also C36.1, C38.1
- net +5V: now also C32.1, C33.1, C34.1, C35.1, C39.1, D10.4 (VDD), D11.2 (A), D5.4 (VDD), D6.4 (VDD), D7.4 (VDD), D8.4 (VDD), D9.4 (VDD), JP1.1 (A), Q2.1 (G), R14.1; no longer J2.A2 (+12V), J2.A3 (+12V), J2.B1 (+12V), J2.B2 (+12V), J2.B3 (+12V)
- net +BATT: now also Q2.3 (D)
- net BUSY: now also U1.13 (GPIO9); no longer U1.3 (GPIO1)
- net CLK1: no longer U1.40 (GPIO26_ADC0)
- net CS1: no longer U1.43 (GPIO29_ADC3)
- net GND: now also C32.2, C33.2, C34.2, C35.2, C36.2, C37.2, C38.2, C39.2, D10.2 (VSS), D5.2 (VSS), D6.2 (VSS), D7.2 (VSS), D8.2 (VSS), D9.2 (VSS), R14.2
- net MISO: now also U1.16 (GPIO12); no longer U1.7 (GPIO4)
- net MISO1: no longer U1.42 (GPIO28_ADC2)
- net MOSI: no longer U1.10 (GPIO7)
- net MOSI1: no longer U1.41 (GPIO27_ADC1)
- net NEOPIXEL_IN: now also U1.40 (GPIO26_ADC0), D8.3 (DIN); no longer U1.27 (GPIO16)
- net SDCS: now also U1.8 (GPIO5); no longer U1.16 (GPIO12)
- net SW1: now also U1.7 (GPIO4); no longer U1.12 (GPIO8)
- net SW2: now also U1.4 (GPIO2); no longer U1.13 (GPIO9)
- net SW3: now also U1.3 (GPIO1); no longer U1.14 (GPIO10)
- net SW4: now also U1.2 (GPIO0); no longer U1.15 (GPIO11)
- net ~{DISCS}: no longer U1.8 (GPIO5)
- net ~{D/C}: now also U1.15 (GPIO11); no longer U1.5 (GPIO3)
- net ~{RES}: now also U1.14 (GPIO10); no longer U1.4 (GPIO2)
- net at U4.19 (VPP): now also C37.1
- net P1 renamed CLK
- net CLK: now also J1.5 (CLK), U4.13 (SCL)
- net P2: no longer names the net of U1.28 (GPIO17)
- net P3: no longer names the net of U1.29 (GPIO18)
- net P7: no longer names the net of U1.31 (GPIO19)
- removed net SCLK: J1.5 (CLK), U1.9 (GPIO6), U4.13 (SCL)
- net SW7: no longer names the net of U1.36 (GPIO24)
- net SW8: no longer names the net of U1.37 (GPIO25)
- new net: D11.1 (K), Q2.2 (S)
- new net: D5.3 (DIN), D8.1 (DOUT)
- new net: D10.3 (DIN), D9.1 (DOUT)
- new net: J2.A2 (+12V), J2.A3 (+12V), J2.B1 (+12V), J2.B2 (+12V), J2.B3 (+12V), JP1.2 (B)
- new net: D5.1 (DOUT), D6.3 (DIN)
- new net: D7.1 (DOUT), D9.3 (DIN)
- new net NEOPIXEL_IN2: D7.3 (DIN), U1.27 (GPIO16)
- no-connect marks 9 -> 10
Other:
- note added: "2.9 inch 3ohm 2.9 inch b/c 0.47R"
- note added: "BS=GND: 4 line SPI"
- note added: "Changelog: Add capacitor to VPP C22 1u -> 100n"
- note added: "Check resistor value for ESR 200 instead of 50"
- note added: "E-Ink Connector"
- note added: "Lipo circuit (unpopulated if budget problems)"
- note added: "Maybe use 10uH instead of 68uH 10k resistor on pin 1 of the mosfet optional"
- note added: "Plug-in connecotr (PCIEx4 compatiable)"
- note added: "Source: Waveshare"
- note added: "USB input"
- note added: "uSD"
- note removed: "C20 & C30 can be removed"
- note removed: "TODO: Ideal diode if there is the budget"
- note removed: "VGL and VGH caps on conn side"
- company: Raspberry Pi Ltd -> Acon (art) & Chengyin Yao (hardware)
- title: RP2350A QFN-60 Minimal Design Example -> Ink screen badge for Undercity
- moved on the sheet: C1, C10, C11, C12, C13, C14, C15, C16, C17, C18, C19, C2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

Commit message: Finish programmer
Parts:
- added JP2: SolderJumper_2_Open, Jumper:SolderJumper-2_P1.3mm_Open_RoundedPad1.0x1.5mm, symbol Jumper:SolderJumper_2_Open
Connections:
- net +3V3: now also JP2.2 (B); no longer J2.A10 (+3.3V), J2.A9 (+3.3V), J2.B10 (3.3Vaux), J2.B8 (+3.3V)
- net CLK1: now also J2.A5 (JTAG2); no longer J2.B19 (PETp1)
- net CS1: now also J2.A8 (JTAG5); no longer J2.B15 (PETn0)
- net MISO1: now also J2.A7 (JTAG4), U1.35 (GPIO23); no longer J2.B14 (PETp0), U1.32 (GPIO20)
- net MOSI1: now also J2.A6 (JTAG3), U1.32 (GPIO20); no longer J2.B20 (PETn1), U1.35 (GPIO23)
- net I2C_CLK: now reaches J2.B5 (SMCLK)
- net I2C_CLK: now also U1.43 (GPIO29_ADC3)
- net I2C_DATA: now reaches J2.B6 (SMDAT)
- net I2C_DATA: now also U1.42 (GPIO28_ADC2)
- new net: J2.A10 (+3.3V), J2.A9 (+3.3V), J2.B10 (3.3Vaux), J2.B8 (+3.3V), JP2.1 (A)
- no-connect marks 10 -> 39
Other:
- note added: "Fixme: Reverse RX/TX"

Commit message: PUSH
Parts:
- removed Q1: Si1308EDL, Package_TO_SOT_SMD:SOT-323_SC-70, symbol Transistor_FET:Si1308EDL
- added C40: 4.7uF, Capacitor_SMD:C_0402_1005Metric, symbol Device:C
- added JP3: SolderJumper_2_Open, Jumper:SolderJumper-2_P1.3mm_Open_RoundedPad1.0x1.5mm, symbol Jumper:SolderJumper_2_Open
- added Q3: IRLML2060, Package_TO_SOT_SMD:SOT-23, symbol Transistor_FET:IRLML2060
- added R11, R15: 470, Resistor_SMD:R_0402_1005Metric, symbol Device:R
- added R16: 33, Resistor_SMD:R_0402_1005Metric, symbol Device:R
- C1, C19, C28, C5, C9: LCSC Part # (none) -> C19702
- C10, C6, C7: LCSC Part # (none) -> C23733
- C11, C12, C13, C14, C15, C16, C17, C18, C2, C22, C32, C33, C34, C35, C36, C8: LCSC Part # (none) -> C1525
- C20, C21, C23, C24, C25, C26, C30, C31, C37, C38: LCSC Part # (none) -> C52923
- C27, C29, C39: LCSC Part # (none) -> C69335
- C3, C4: LCSC Part # (none) -> C1548
- D1, D11, D2, D3: LCSC Part # (none) -> C5204746
- D10, D5, D6, D7, D8, D9: LCSC Part # C965555 -> C5349955
- D4: LCSC Part # (none) -> C2286
- H1, H2, H3, H4: symbol Mechanical:MountingHole -> Mechanical:MountingHole_Pad
- J2, J5: now left out of the parts list
- L1: LCSC Part # (none) -> C42411119
- L2: footprint Inductor_SMD:L_Ferrocore_DLG-0403 -> Inductor_SMD:L_APV_ANR4018; LCSC Part # C2929419 -> C167808
- Q2: LCSC Part # (none) -> C15127
- R1, R13: LCSC Part # (none) -> C25744
- R10, R14: LCSC Part # (none) -> C25867
- R12: value 3 -> 0.47; LCSC Part # (none) -> C3017627
- R2, R4, R6: LCSC Part # (none) -> C11702
- R3, R5: LCSC Part # (none) -> C25905
- R7, R8: LCSC Part # (none) -> C25105
- R9: value 5k -> 5.1k; LCSC Part # (none) -> C25905
- SW1, SW2: footprint Button_Switch_SMD:SW_SPST_B3U-1000P -> inkbadge:SW_Push_SPST_TSA016; LCSC Part # (none) -> C2888430
- U1: LCSC Part # (none) -> C42411118
- U2: LCSC Part # (none) -> C6186
- U3: LCSC Part # (none) -> C85364
- U4: LCSC Part # (none) -> C262567
- U5: LCSC Part # (none) -> C97521
- U6: LCSC Part # (none) -> C16581
- Y1: footprint Crystal:Crystal_SMD_2520-4Pin_2.5x2.0mm -> Crystal:Crystal_SMD_3225-4Pin_3.2x2.5mm; LCSC Part # C7301971 -> C20625731
Connections:
- net +3V3: now also R16.1
- net +5V: now also D11.1 (K), Q2.2 (S), JP3.2 (B); no longer C9.1, D11.2 (A), D4.2 (A), J3.A4 (VBUS), J3.A9 (VBUS), J3.B4 (VBUS), J3.B9 (VBUS), Q2.1 (G), R14.1, U3.5 (VP), U6.4 (V_{CC}), U6.8 (CE)
- net GDR: now also Q3.1 (G)
- net GND: now also H1.1, H2.1, H3.1, H4.1, C40.2
- net NEOPIXEL_IN: now also U1.41 (GPIO27_ADC1), R11.1; no longer D8.3 (DIN), U1.40 (GPIO26_ADC0)
- net NEOPIXEL_IN2: now also R15.1; no longer D7.3 (DIN)
- net RESE: now also Q3.2 (S)
- net at C27.2, D3.2 (A), L2.2: now also Q3.3 (D)
- net at U1.46 (VREG_AVDD): now also C40.1, R16.2
- new net: D7.3 (DIN), R15.2
- new net: D8.3 (DIN), R11.2
- new net VBUS: C9.1, D11.2 (A), D4.2 (A), J3.A4 (VBUS), J3.A9 (VBUS), J3.B4 (VBUS), J3.B9 (VBUS), JP3.1 (A), Q2.1 (G), R14.1, U3.5 (VP), U6.4 (V_{CC}), U6.8 (CE)
- no-connect marks 39 -> 47
Other:
- note added: "Maybe use 68uH instead of 10uH 10k resistor on pin 1 of the mosfet optional"
- note added: "Plug-in connector (PCIEx4 compatiable)"
- note removed: "Check resistor value for ESR 200 instead of 50"
- note removed: "Fixme: Reverse RX/TX"
- note removed: "Maybe use 10uH instead of 68uH 10k resistor on pin 1 of the mosfet optional"
- note removed: "Plug-in connecotr (PCIEx4 compatiable)"
- company: Acon (art) & Chengyin Yao (hardware) -> Acon (design) & Bunnyguy (art) & Cyao (hardware)
- moved on the sheet: C2, C20, C21, C22, C23, C24, C25, C26, C30, C31, C32, C33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

Commit message: SOME FIRMWARE IG FAQ THE WORLD IDC ME DIE
Parts:
- C40: LCSC Part # C1548 -> C23733
Changed lines of the file:
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@@
 			)
 		)
-		(property "LCSC Part #" "C1548"
+		(property "LCSC Part #" "C23733"
 			(at 134.62 49.53 0)
 			(effects
