File: inkbadge/inkbadge.kicad_sch (KiCad schematic)
At the start: 95 parts, among them J1 Micro_SD_Card, J2 Bus_PCI_Express_x4, J3 USB_C_Receptacle_USB2.0_14P, J5 Conn_01x02, Q2 AO3401A, Q3 IRLML2060, SW1 SW_Push, SW2 SW_Push, SW3 SW_Push, SW4 SW_Push, SW5 SW_Push, SW6 SW_Push, U1 RP2350A, U2 NCP1117-3.3_SOT223, U3 SRV05-4, U4 Conn, U5 W25Q128JVS, U6 TP4056-42-ESOP8, Y1 12MHz 10pf

Commit message: FIRMWARE IDKFHRGVKQHBJ
Changed lines of the file:
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@@
 	(wire
 		(pts
-			(xy 213.36 124.46) (xy 220.98 124.46)
+			(xy 213.36 124.46) (xy 227.33 124.46)
 		)
 		(stroke
@@
 	(wire
 		(pts
-			(xy 213.36 93.98) (xy 220.98 93.98)
+			(xy 213.36 93.98) (xy 227.33 93.98)
 		)
 		(stroke
@@
 	(wire
 		(pts
-			(xy 213.36 68.58) (xy 220.98 68.58)
+			(xy 213.36 68.58) (xy 227.33 68.58)
 		)
 		(stroke
@@
 	(wire
 		(pts
-			(xy 213.36 78.74) (xy 220.98 78.74)
+			(xy 213.36 78.74) (xy 227.33 78.74)
 		)
 		(stroke
@@
 	(wire
 		(pts
-			(xy 220.98 101.6) (xy 213.36 101.6)
+			(xy 227.33 101.6) (xy 213.36 101.6)
 		)
 		(stroke
@@
 	(wire
 		(pts
-			(xy 213.36 66.04) (xy 220.98 66.04)
+			(xy 213.36 66.04) (xy 227.33 66.04)
 		)
 		(stroke
@@
 	(wire
 		(pts
-			(xy 213.36 116.84) (xy 220.98 116.84)
+			(xy 213.36 116.84) (xy 227.33 116.84)
 		)
 		(stroke
@@
 	(wire
 		(pts
-			(xy 220.98 104.14) (xy 213.36 104.14)
+			(xy 227.33 104.14) (xy 213.36 104.14)
 		)
 		(stroke
@@
 	(wire
 		(pts
-			(xy 220.98 99.06) (xy 213.36 99.06)
+			(xy 227.33 99.06) (xy 213.36 99.06)
 		)
 		(stroke
@@
 	(wire
 		(pts
-			(xy 220.98 96.52) (xy 213.36 96.52)
+			(xy 227.33 96.52) (xy 213.36 96.52)
 		)
 		(stroke
@@
 	(wire
 		(pts
-			(xy 213.36 76.2) (xy 220.98 76.2)
+			(xy 213.36 76.2) (xy 227.33 76.2)
 		)
 		(stroke
@@
 	(wire
 		(pts
-			(xy 67.31 149.86) (xy 77.47 149.86)
+			(xy 67.31 149.86) (xy 76.2 149.86)
 		)
 		(stroke
@@
 	(wire
 		(pts
-			(xy 213.36 71.12) (xy 220.98 71.12)
+			(xy 213.36 71.12) (xy 227.33 71.12)
 		)
 		(stroke
@@
 	(wire
 		(pts
-			(xy 213.36 88.9) (xy 220.98 88.9)
+			(xy 213.36 88.9) (xy 227.33 88.9)
 		)
 		(stroke
@@
 	(wire
 		(pts
-			(xy 45.72 139.7) (xy 77.47 139.7)
+			(xy 45.72 139.7) (xy 76.2 139.7)
 		)
 		(stroke
@@
 	(wire
 		(pts
-			(xy 213.36 91.44) (xy 220.98 91.44)
+			(xy 213.36 91.44) (xy 227.33 91.44)
 		)
 		(stroke
@@
 	(wire
 		(pts
-			(xy 213.36 121.92) (xy 220.98 121.92)
+			(xy 213.36 121.92) (xy 227.33 121.92)
 		)
 		(stroke
@@
 	(wire
 		(pts
-			(xy 213.36 119.38) (xy 220.98 119.38)
+			(xy 213.36 119.38) (xy 227.33 119.38)
 		)
 		(stroke
@@
 	)
 	(label "MOSI1"
-		(at 220.98 116.84 180)
+		(at 227.33 116.84 180)
 		(effects
 			(font
@@
 	)
 	(label "BUSY"
-		(at 220.98 88.9 180)
+		(at 227.33 88.9 180)
 		(effects
 			(font
@@
 	)
 	(label "SW2"
-		(at 220.98 71.12 180)
+		(at 227.33 71.12 180)
 		(effects
 			(font
@@
 	)
 	(label "SW3"
-		(at 220.98 68.58 180)
+		(at 227.33 68.58 180)
 		(effects
 			(font
@@
 	)
 	(label "~{D{slash}C}"
-		(at 220.98 93.98 180)
+		(at 227.33 93.98 180)
 		(effects
 			(font
@@
 	)
 	(label "XOUT"
-		(at 77.47 149.86 180)
+		(at 76.2 149.86 180)
 		(effects
 			(font
@@
 	)
 	(label "MISO1"
-		(at 220.98 124.46 180)
+		(at 227.33 124.46 180)
 		(effects
 			(font
@@
 	)
 	(label "MISO"
-		(at 220.98 96.52 180)
+		(at 227.33 96.52 180)
 		(effects
 			(font
@@
 	)
 	(label "CS1"
-		(at 220.98 119.38 180)
+		(at 227.33 119.38 180)
 		(effects
 			(font
@@
 	)
 	(label "XIN"
-		(at 77.47 139.7 180)
+		(at 76.2 139.7 180)
 		(effects
 			(font
@@
 	)
 	(label "SDCS"
-		(at 220.98 78.74 180)
+		(at 227.33 78.74 180)
 		(effects
 			(font
@@
 	)
 	(label "SW4"
-		(at 220.98 66.04 180)
+		(at 227.33 66.04 180)
 		(effects
 			(font
@@
 	)
 	(label "SW1"
-		(at 220.98 76.2 180)
+		(at 227.33 76.2 180)
 		(effects
 			(font
@@
 	)
 	(label "MOSI"
-		(at 220.98 104.14 180)
+		(at 227.33 104.14 180)
 		(effects
 			(font
@@
 	)
 	(label "~{DISCS}"
-		(at 220.98 99.06 180)
+		(at 227.33 99.06 180)
 		(effects
 			(font
@@
 	)
 	(label "~{RES}"
-		(at 220.98 91.44 180)
+		(at 227.33 91.44 180)
 		(effects
 			(font
@@
 	)
 	(label "CLK1"
-		(at 220.98 121.92 180)
+		(at 227.33 121.92 180)
 		(effects
 			(font
@@
 	)
 	(label "CLK"
-		(at 220.98 101.6 180)
+		(at 227.33 101.6 180)
 		(effects
 			(font
